Commit message: Wheels are now turning. Steps towards simulation.

File: kymco_maxxer90_description/urdf/front_wheel.urdf.xacro (robot description, xacro)
@@ -22,20 +22,32 @@
 			</collision>
 		</link>
+        <link name="${wheel_prefix}_wheel_steering_link" />
+        <joint name="${wheel_prefix}_steering_wheel_joint" type="revolute">
+			<xacro:insert_block name="joint_pose"/>
+			<parent link="base_link"/>
+			<child link="${wheel_prefix}_wheel_steering_link"/>
+            <axis xyz="0 0 1" />
+            <mimic joint="steering_wheel_joint" multiplier="1" offset="0" />
+            <!-- TODO effort and velocity -->
+            <limit lower="${-PI*25/180}" upper="${PI*25/180}" effort="0.5" velocity="4.5"/>
+            <dynamics damping="0.02" friction="0.0" />
+        </joint>
 		<joint name="${wheel_prefix}_wheel" type="continuous">
-			<parent link="steering_wheel_link"/>
+            <origin xyz="0 0 0" />
+            <parent link="${wheel_prefix}_wheel_steering_link" />
 			<child link="${wheel_prefix}_wheel_link"/>
-			<xacro:insert_block name="joint_pose"/>
 			<axis xyz="0 1 0" rpy="0 0 0" />
-		</joint>
-        <!-- TODO plugins for ackermann steering-->
-        <!-- <transmission name="${wheel_prefix}_wheel_trans" type="SimpleTransmission"> -->
-            <!-- <type>transmission_interface/SimpleTransmission</type> -->
-            <!-- <actuator name="${wheel_prefix}_wheel_motor"> -->
-                <!-- <mechanicalReduction>1</mechanicalReduction> -->
-            <!-- </actuator> -->
-            <!-- <joint name="${wheel_prefix}_wheel"> -->
-                <!-- <hardwareInterface>VelocityJointInterface</hardwareInterface> -->
-            <!-- </joint> -->
-        <!-- </transmission> -->
+        </joint>
+        <gazebo>
+            <plugin name="${wheel_prefix}_mimic_joint_plugin" filename="libroboticsgroup_gazebo_mimic_joint_plugin.so">
+                <joint>steering_wheel_joint</joint>
+                <mimicJoint>${wheel_prefix}_steering_wheel_joint</mimicJoint>
+                <hasPID/>
+                <multiplier>1.0</multiplier>
+                <offset>0</offset>
+                <sensitiveness></sensitiveness>
+                <maxEffort>10.0</maxEffort>
+            </plugin>
+        </gazebo>
 	</xacro:macro>
 </robot>

File: kymco_maxxer90_description/urdf/kymco_maxxer90.urdf.xacro (robot description, xacro)
@@ -9,4 +9,5 @@
     <xacro:property name="wheel_width" value="0.15"/>
     <xacro:property name="track" value="0.55"/>
+    <!-- Chassis -->
     <link name="base_link">
         <visual>
@@ -26,4 +27,5 @@
         </collision>
     </link>
+    <!-- Steering wheel -->
     <link name="steering_wheel_link"/>
     <joint name="steering_wheel_joint" type="revolute">
@@ -35,4 +37,14 @@
         <limit lower="${-PI*25/180}" upper="${PI*25/180}" effort="0.5" velocity="4.5"/>
     </joint>
+    <transmission name="steering_wheel_joint_trans">
+        <type>transmission_interface/SimpleTransmission</type>
+        <joint name="steering_wheel_joint">
+            <hardwareInterface>hardware_interface/PositionJointInterface</hardwareInterface>
+        </joint>
+        <actuator name="steering_wheel_actuator">
+            <mechanicalReduction>1</mechanicalReduction>
+        </actuator>
+    </transmission>
+    <!-- Engine -->
     <link name="engine_link">
         <visual>
@@ -57,4 +69,5 @@
         <child link="engine_link" />
     </joint>
+    <!-- Wheels -->
     <xacro:kymco_maxxer90_front_wheel wheel_prefix="front_right">
         <origin xyz="${track/2} 0.33 ${distance_from_ground/2}" rpy="0 0 ${PI/2}"/>

File: kymco_maxxer90_description/urdf/wheel.urdf.xacro (robot description, xacro)
@@ -28,14 +28,13 @@
 			<axis xyz="0 1 0" rpy="0 0 0" />
 		</joint>
-        <!-- TODO plugins for ackermann steering-->
-        <!-- <transmission name="${wheel_prefix}_wheel_trans" type="SimpleTransmission"> -->
-            <!-- <type>transmission_interface/SimpleTransmission</type> -->
-            <!-- <actuator name="${wheel_prefix}_wheel_motor"> -->
-                <!-- <mechanicalReduction>1</mechanicalReduction> -->
-            <!-- </actuator> -->
-            <!-- <joint name="${wheel_prefix}_wheel"> -->
-                <!-- <hardwareInterface>VelocityJointInterface</hardwareInterface> -->
-            <!-- </joint> -->
-        <!-- </transmission> -->
+        <transmission name="${wheel_prefix}_wheel_trans" type="SimpleTransmission">
+            <type>transmission_interface/SimpleTransmission</type>
+            <actuator name="${wheel_prefix}_wheel_motor">
+                <mechanicalReduction>1</mechanicalReduction>
+            </actuator>
+            <joint name="${wheel_prefix}_wheel">
+                <hardwareInterface>VelocityJointInterface</hardwareInterface>
+            </joint>
+        </transmission>
 	</xacro:macro>
 </robot>

Commit message: Fixes towards proper simulation. The model can now properly turn. I need to check self collisions.

File: kymco_maxxer90_description/urdf/front_wheel.urdf.xacro (robot description, xacro)
@@ -3,9 +3,10 @@
 	<xacro:macro name="kymco_maxxer90_front_wheel" params="wheel_prefix *joint_pose">
 		<link name="${wheel_prefix}_wheel_link">
-			<inertial>
-				<mass value="5.0" />  <!-- TODO -->
-				<origin xyz="0 0 0" />
-				<inertia  ixx="0.02467" ixy="0" ixz="0" iyy="0.02467" iyz="0" izz="0.04411" />  <!-- TODO -->
-			</inertial>
+            <!-- TODO -->
+            <inertial>
+                <mass value="33.455"/>
+                <origin xyz="-0.08748 -0.00085 0.09947"/>
+                <inertia ixx="0.6022" ixy="-0.02364" ixz="-0.1197" iyy="1.7386" iyz="-0.001544" izz="2.0296"/>
+            </inertial>
 			<visual>
 				<origin xyz="0 0 0" rpy="0 0 0" />
@@ -22,5 +23,12 @@
 			</collision>
 		</link>
-        <link name="${wheel_prefix}_wheel_steering_link" />
+        <link name="${wheel_prefix}_wheel_steering_link" >
+            <!-- TODO -->
+            <inertial>
+                <mass value="33.455"/>
+                <origin xyz="-0.08748 -0.00085 0.09947"/>
+                <inertia ixx="0.6022" ixy="-0.02364" ixz="-0.1197" iyy="1.7386" iyz="-0.001544" izz="2.0296"/>
+            </inertial>
+        </link>
         <joint name="${wheel_prefix}_steering_wheel_joint" type="revolute">
 			<xacro:insert_block name="joint_pose"/>

File: kymco_maxxer90_description/urdf/kymco_maxxer90.urdf.xacro (robot description, xacro)
@@ -11,4 +11,10 @@
     <!-- Chassis -->
     <link name="base_link">
+        <!-- TODO -->
+        <inertial>
+            <mass value="129"/>
+            <origin xyz="-0.08748 -0.00085 0.09947"/>
+            <inertia ixx="0.6022" ixy="-0.02364" ixz="-0.1197" iyy="1.7386" iyz="-0.001544" izz="2.0296"/>
+        </inertial>
         <visual>
             <origin xyz="0 0 ${distance_from_ground}" rpy="0 0 0"/>
@@ -28,5 +34,12 @@
     </link>
     <!-- Steering wheel -->
-    <link name="steering_wheel_link"/>
+    <link name="steering_wheel_link">
+        <!-- TODO -->
+        <inertial>
+            <mass value="3.5"/>
+            <origin xyz="-0.08748 -0.00085 0.09947"/>
+            <inertia ixx="0.6022" ixy="-0.02364" ixz="-0.1197" iyy="1.7386" iyz="-0.001544" izz="2.0296"/>
+        </inertial>
+    </link>
     <joint name="steering_wheel_joint" type="revolute">
         <origin xyz="0 0 0" rpy="0 0 0" />
@@ -36,4 +49,5 @@
         <!-- TODO effort and velocity -->
         <limit lower="${-PI*25/180}" upper="${PI*25/180}" effort="0.5" velocity="4.5"/>
+        <dynamics damping="0.02" friction="0.0" />
     </joint>
     <transmission name="steering_wheel_joint_trans">

Commit message: Trying (and failing) to have accurately simulate the quad

File: kymco_maxxer90_description/urdf/front_wheel.urdf.xacro (robot description, xacro)
@@ -3,9 +3,8 @@
 	<xacro:macro name="kymco_maxxer90_front_wheel" params="wheel_prefix *joint_pose">
 		<link name="${wheel_prefix}_wheel_link">
-            <!-- TODO -->
             <inertial>
-                <mass value="33.455"/>
+                <mass value="15.0"/>
                 <origin xyz="-0.08748 -0.00085 0.09947"/>
-                <inertia ixx="0.6022" ixy="-0.02364" ixz="-0.1197" iyy="1.7386" iyz="-0.001544" izz="2.0296"/>
+                <inertia  ixx="0.28813432952881635" ixy="0" ixz="0" iyy="0.5212991167201597" iyz="0" izz="0.2894147916616918" />
             </inertial>
 			<visual>
@@ -24,9 +23,8 @@
 		</link>
         <link name="${wheel_prefix}_wheel_steering_link" >
-            <!-- TODO -->
             <inertial>
-                <mass value="33.455"/>
+                <mass value="0.01"/>
                 <origin xyz="-0.08748 -0.00085 0.09947"/>
-                <inertia ixx="0.6022" ixy="-0.02364" ixz="-0.1197" iyy="1.7386" iyz="-0.001544" izz="2.0296"/>
+                <inertia ixx="0.0000001" ixy="0" ixz="0" iyy="0.0000001" iyz="0" izz="0.0000001"/>
             </inertial>
         </link>
@@ -47,4 +45,7 @@
 			<axis xyz="0 1 0" rpy="0 0 0" />
         </joint>
+        <gazebo reference="${wheel_prefix}_wheel_link">
+            <material>Gazebo/Black</material>
+        </gazebo>"
         <gazebo>
             <plugin name="${wheel_prefix}_mimic_joint_plugin" filename="libroboticsgroup_gazebo_mimic_joint_plugin.so">

File: kymco_maxxer90_description/urdf/kymco_maxxer90.urdf.xacro (robot description, xacro)
@@ -10,10 +10,10 @@
     <xacro:property name="track" value="0.55"/>
     <!-- Chassis -->
-    <link name="base_link">
-        <!-- TODO -->
+    <link name="base_link" />
+    <link name="chassis_link">
         <inertial>
-            <mass value="129"/>
+            <mass value="68"/>
             <origin xyz="-0.08748 -0.00085 0.09947"/>
-            <inertia ixx="0.6022" ixy="-0.02364" ixz="-0.1197" iyy="1.7386" iyz="-0.001544" izz="2.0296"/>
+                <inertia  ixx="2.746671789898144" ixy="0" ixz="0" iyy="1.629571305145487" iyz="0" izz="1.930434142335272" />
         </inertial>
         <visual>
@@ -33,11 +33,18 @@
         </collision>
     </link>
+    <joint name="chassis_joint" type="fixed">
+        <origin xyz="0 0 0" rpy="0 0 0" />
+        <parent link="base_link" />"
+        <child link="chassis_link" />"
+    </joint>
+    <gazebo reference="chassis_link">
+        <material>Gazebo/Black</material>
+    </gazebo>"
     <!-- Steering wheel -->
     <link name="steering_wheel_link">
-        <!-- TODO -->
         <inertial>
-            <mass value="3.5"/>
+            <mass value="0.1"/>
             <origin xyz="-0.08748 -0.00085 0.09947"/>
-            <inertia ixx="0.6022" ixy="-0.02364" ixz="-0.1197" iyy="1.7386" iyz="-0.001544" izz="2.0296"/>
+            <inertia ixx="0.0000001" ixy="0" ixz="0" iyy="0.0000001" iyz="-0" izz="0.0000001"/>
         </inertial>
     </link>
@@ -83,4 +90,7 @@
         <child link="engine_link" />
     </joint>
+    <gazebo reference="engine_link">
+        <material>Gazebo/Grey</material>
+    </gazebo>"
     <!-- Wheels -->
     <xacro:kymco_maxxer90_front_wheel wheel_prefix="front_right">
@@ -116,4 +126,7 @@
         <child link="rear_axle_link" />
     </joint>
+    <gazebo reference="rear_axle_link">
+        <material>Gazebo/Grey</material>
+    </gazebo>"
     <link name="front_plate_link">
         <visual>
@@ -136,4 +149,7 @@
         <child link="front_plate_link" />
     </joint>
+    <gazebo reference="front_plate_link">
+        <material>Gazebo/Grey</material>
+    </gazebo>"
     <link name="rear_plate_link">
         <visual>
@@ -156,4 +172,7 @@
         <child link="rear_plate_link" />
     </joint>
+    <gazebo reference="rear_plate_link">
+        <material>Gazebo/Grey</material>
+    </gazebo>"
     <link name="rear_trans_chassis_link">
         <visual>
@@ -176,4 +195,7 @@
         <child link="rear_trans_chassis_link" />
     </joint>
+    <gazebo reference="rear_trans_chassis_link">
+        <material>Gazebo/Black</material>
+    </gazebo>"
     <link name="rear_trans_link">
         <visual>
@@ -196,4 +218,7 @@
         <child link="rear_trans_link" />
     </joint>
+    <gazebo reference="rear_trans_link">
+        <material>Gazebo/Black</material>
+    </gazebo>"
     <link name="rear_trans_spring_link">
         <visual>
@@ -213,4 +238,7 @@
         </collision>
     </link>
+    <gazebo reference="rear_trans_spring_link">
+        <material>Gazebo/Red</material>
+    </gazebo>"
     <joint name="rear_trans_spring_joint" type="fixed">
         <origin xyz="0 -0.56 0.29" rpy="${-PI/4} 0 0"/>
@@ -238,4 +266,7 @@
         <child link="front_right_trans_chassis_link" />
     </joint>
+    <gazebo reference="front_right_trans_chassis_link">
+        <material>Gazebo/Black</material>
+    </gazebo>"
     <link name="front_right_trans_link">
         <visual>
@@ -258,4 +289,7 @@
         <child link="front_right_trans_link" />
     </joint>
+    <gazebo reference="front_right_trans_link">
+        <material>Gazebo/Black</material>
+    </gazebo>"
     <link name="front_right_trans_spring_link">
         <visual>
@@ -280,4 +314,7 @@
         <child link="front_right_trans_spring_link" />
     </joint>
+    <gazebo reference="front_right_trans_spring_link">
+        <material>Gazebo/Red</material>
+    </gazebo>"
     <link name="front_left_trans_chassis_link">
         <visual>
@@ -300,4 +337,7 @@
         <child link="front_left_trans_chassis_link" />
     </joint>
+    <gazebo reference="front_left_trans_chassis_link">
+        <material>Gazebo/Black</material>
+    </gazebo>"
     <link name="front_left_trans_link">
         <visual>
@@ -320,4 +360,7 @@
         <child link="front_left_trans_link" />
     </joint>
+    <gazebo reference="front_left_trans_link">
+        <material>Gazebo/Black</material>
+    </gazebo>"
     <link name="front_left_trans_spring_link">
         <visual>
@@ -342,3 +385,6 @@
         <child link="front_left_trans_spring_link" />
     </joint>
+    <gazebo reference="front_left_trans_spring_link">
+        <material>Gazebo/Red</material>
+    </gazebo>"
 </robot>

File: kymco_maxxer90_description/urdf/wheel.urdf.xacro (robot description, xacro)
@@ -4,7 +4,7 @@
 		<link name="${wheel_prefix}_wheel_link">
 			<inertial>
-				<mass value="5.0" />  <!-- TODO -->
-				<origin xyz="0 0 0" />
-				<inertia  ixx="0.02467" ixy="0" ixz="0" iyy="0.02467" iyz="0" izz="0.04411" />  <!-- TODO -->
+				<mass value="15.0" />
+                <origin xyz="0 0 0" />
+                <inertia  ixx="0.28813432952881635" ixy="0" ixz="0" iyy="0.5212991167201597" iyz="0" izz="0.2894147916616918" />
 			</inertial>
 			<visual>
@@ -28,4 +28,7 @@
 			<axis xyz="0 1 0" rpy="0 0 0" />
 		</joint>
+        <gazebo reference="${wheel_prefix}_wheel_link">
+            <material>Gazebo/Black</material>
+        </gazebo>"
         <transmission name="${wheel_prefix}_wheel_trans" type="SimpleTransmission">
             <type>transmission_interface/SimpleTransmission</type>
