Commit message: Various description fixed. Current problems: Inertia and mimic joints in Gazebo

File: kymco_maxxer90_description/urdf/front_wheel.urdf.xacro (robot description, xacro)
@@ -5,5 +5,5 @@
             <inertial>
                 <mass value="15.0"/>
-                <origin xyz="-0.08748 -0.00085 0.09947"/>
+                <origin xyz="0 0 0"/>
                 <inertia  ixx="0.28813432952881635" ixy="0" ixz="0" iyy="0.5212991167201597" iyz="0" izz="0.2894147916616918" />
             </inertial>
@@ -24,7 +24,7 @@
         <link name="${wheel_prefix}_wheel_steering_link" >
             <inertial>
-                <mass value="0.01"/>
-                <origin xyz="-0.08748 -0.00085 0.09947"/>
-                <inertia ixx="0.0000001" ixy="0" ixz="0" iyy="0.0000001" iyz="0" izz="0.0000001"/>
+                <mass value="1"/>
+                <origin xyz="0 0 0"/>
+                <inertia ixx="0.01" ixy="0" ixz="0" iyy="0.01" iyz="0" izz="0.01"/>
             </inertial>
         </link>
@@ -36,9 +36,9 @@
             <mimic joint="steering_wheel_joint" multiplier="1" offset="0" />
             <!-- TODO effort and velocity -->
-            <limit lower="${-PI*25/180}" upper="${PI*25/180}" effort="0.5" velocity="4.5"/>
-            <dynamics damping="0.02" friction="0.0" />
+            <limit lower="${-PI*25/180}" upper="${PI*25/180}" effort="100.5" velocity="4.5"/>
+            <dynamics damping="0.2" friction="0" />
         </joint>
 		<joint name="${wheel_prefix}_wheel" type="continuous">
-            <origin xyz="0 0 0" />
+            <origin xyz="0 0 0" rpy="0 0 0"/>
             <parent link="${wheel_prefix}_wheel_steering_link" />
 			<child link="${wheel_prefix}_wheel_link"/>
@@ -55,8 +55,26 @@
                 <multiplier>1.0</multiplier>
                 <offset>0</offset>
-                <sensitiveness></sensitiveness>
+                <sensitiveness>0.0</sensitiveness>
                 <maxEffort>10.0</maxEffort>
             </plugin>
         </gazebo>
+        <!-- <transmission name="${wheel_prefix}_wheel_steering_joint_trans"> -->
+            <!-- <type>transmission_interface/SimpleTransmission</type> -->
+            <!-- <joint name="${wheel_prefix}_steering_wheel_joint"> -->
+                <!-- <hardwareInterface>hardware_interface/PositionJointInterface</hardwareInterface> -->
+            <!-- </joint> -->
+            <!-- <actuator name="${wheel_prefix}_steering_wheel_actuator"> -->
+                <!-- <mechanicalReduction>1</mechanicalReduction> -->
+            <!-- </actuator> -->
+        <!-- </transmission> -->
+        <!-- <transmission name="${wheel_prefix}_wheel_trans" type="SimpleTransmission"> -->
+            <!-- <type>transmission_interface/SimpleTransmission</type> -->
+            <!-- <actuator name="${wheel_prefix}_wheel_motor"> -->
+                <!-- <mechanicalReduction>0</mechanicalReduction> -->
+            <!-- </actuator> -->
+            <!-- <joint name="${wheel_prefix}_wheel"> -->
+                <!-- <hardwareInterface>hardware_interface/VelocityJointInterface</hardwareInterface> -->
+            <!-- </joint> -->
+        <!-- </transmission> -->
 	</xacro:macro>
 </robot>

File: kymco_maxxer90_description/urdf/kymco_maxxer90.urdf.xacro (robot description, xacro)
@@ -36,5 +36,5 @@
         <inertial>
             <mass value="68"/>
-            <origin xyz="0 0.2 0.37"/>
+            <origin xyz="0 -0.2 0.37"/>
                 <inertia  ixx="11.746671789898144" ixy="0" ixz="0" iyy="2.629571305145487" iyz="0" izz="10.930434142335272" />
         </inertial>
@@ -51,7 +51,7 @@
     <link name="steering_wheel_link">
         <inertial>
-            <mass value="0.1"/>
-            <origin xyz="-0.08748 -0.00085 0.09947"/>
-            <inertia ixx="0.0000001" ixy="0" ixz="0" iyy="0.0000001" iyz="-0" izz="0.0000001"/>
+            <mass value="1"/>
+            <origin xyz="0 0 0"/>
+            <inertia ixx="0.01" ixy="0" ixz="0" iyy="0.01" iyz="0" izz="0.01"/>
         </inertial>
     </link>
@@ -62,6 +62,6 @@
         <axis xyz="0 0 1" />
         <!-- TODO effort and velocity -->
-        <limit lower="${-PI*25/180}" upper="${PI*25/180}" effort="0.5" velocity="4.5"/>
-        <dynamics damping="0.02" friction="0.0" />
+        <limit lower="${-PI*25/180}" upper="${PI*25/180}" effort="100.5" velocity="4.5"/>
+        <dynamics damping="20" friction="2.0" />
     </joint>
     <transmission name="steering_wheel_joint_trans">
@@ -85,10 +85,10 @@
             </material>
         </visual>
-        <!-- <collision> -->
-            <!-- <origin xyz="0 0 0" rpy="0 0 0"/> -->
-            <!-- <geometry> -->
-                <!-- <mesh filename="package://kymco_maxxer90_description/meshes/engine.stl" scale="1.0 1.0 1.0"/> -->
-            <!-- </geometry> -->
-        <!-- </collision> -->
+        <collision>
+            <origin xyz="0 0 0" rpy="0 0 0"/>
+            <geometry>
+                <mesh filename="package://kymco_maxxer90_description/meshes/engine.stl" scale="1.0 1.0 1.0"/>
+            </geometry>
+        </collision>
     </link>
     <joint name="engine_joint" type="fixed">
@@ -101,16 +101,16 @@
     </gazebo>"
     <!-- Wheels -->
-    <!-- <xacro:kymco_maxxer90_front_wheel wheel_prefix="front_right"> -->
-        <!-- <origin xyz="${track/2} 0.33 ${distance_from_ground/2}" rpy="0 0 ${PI/2}"/> -->
-    <!-- </xacro:kymco_maxxer90_front_wheel> -->
-    <!-- <xacro:kymco_maxxer90_front_wheel wheel_prefix="front_left"> -->
-        <!-- <origin xyz="${-track/2} 0.33 ${distance_from_ground/2}" rpy="0 0 ${-PI/2}"/> -->
-    <!-- </xacro:kymco_maxxer90_front_wheel> -->
-    <!-- <xacro:kymco_maxxer90_wheel wheel_prefix="rear_left"> -->
-        <!-- <origin xyz="${-track/2} ${0.33-wheelbase} ${distance_from_ground/2}" rpy="0 0 ${-PI/2}"/> -->
-    <!-- </xacro:kymco_maxxer90_wheel> -->
-    <!-- <xacro:kymco_maxxer90_wheel wheel_prefix="rear_right"> -->
-        <!-- <origin xyz="${track/2} ${0.33-wheelbase} ${distance_from_ground/2}" rpy="0 0 ${PI/2}"/> -->
-    <!-- </xacro:kymco_maxxer90_wheel> -->
+    <xacro:kymco_maxxer90_front_wheel wheel_prefix="front_right">
+        <origin xyz="${track/2} 0.33 ${distance_from_ground/2}" rpy="0 0 ${PI/2}"/>
+    </xacro:kymco_maxxer90_front_wheel>
+    <xacro:kymco_maxxer90_front_wheel wheel_prefix="front_left">
+        <origin xyz="${-track/2} 0.33 ${distance_from_ground/2}" rpy="0 0 ${-PI/2}"/>
+    </xacro:kymco_maxxer90_front_wheel>
+    <xacro:kymco_maxxer90_wheel wheel_prefix="rear_left">
+        <origin xyz="${-track/2} 0 0" rpy="0 0 ${-PI/2}"/>
+    </xacro:kymco_maxxer90_wheel>
+    <xacro:kymco_maxxer90_wheel wheel_prefix="rear_right">
+        <origin xyz="${track/2} 0 0" rpy="0 0 ${PI/2}"/>
+    </xacro:kymco_maxxer90_wheel>
     <link name="rear_axle_link">
         <visual>
@@ -121,10 +121,10 @@
             <material name="silver"/>
         </visual>
-        <!-- <collision> -->
-            <!-- <origin xyz="0 0 0" rpy="0 0 0"/> -->
-            <!-- <geometry> -->
-                <!-- <mesh filename="package://kymco_maxxer90_description/meshes/differential.stl" scale="1.0 1.0 1.0"/> -->
-            <!-- </geometry> -->
-        <!-- </collision> -->
+        <collision>
+            <origin xyz="0 0 0" rpy="0 0 0"/>
+            <geometry>
+                <mesh filename="package://kymco_maxxer90_description/meshes/differential.stl" scale="1.0 1.0 1.0"/>
+            </geometry>
+        </collision>
     </link>
     <joint name="rear_axle_joint" type="fixed">
@@ -135,5 +135,27 @@
     <gazebo reference="rear_axle_link">
         <material>Gazebo/Grey</material>
-    </gazebo>"
+    </gazebo>
+    <link name="RWD">
+        <inertial>
+            <mass value="1"/>
+            <origin xyz="0 0 0"/>
+            <inertia ixx="0.01" ixy="0" ixz="0" iyy="0.01" iyz="0" izz="0.01"/>
+        </inertial>
+    </link>
+    <joint name="RWD_joint" type="continuous">
+        <origin xyz="0 ${0.33-wheelbase} ${distance_from_ground/2}" rpy="0 0 0"/>
+        <parent link="base_link" />
+        <child link="RWD" />
+        <axis xyz="-1 0 0" />
+    </joint>
+    <transmission name="non_differential_trans" type="SimpleTransmission">
+        <type>transmission_interface/SimpleTransmission</type>
+        <actuator name="non_differential_motor">
+            <mechanicalReduction>1</mechanicalReduction>
+        </actuator>
+        <joint name="RWD_joint">
+            <hardwareInterface>hardware_interface/VelocityJointInterface</hardwareInterface>
+        </joint>
+    </transmission>
     <link name="front_plate_link">
         <visual>
@@ -144,10 +166,10 @@
             <material name="silver"/>
         </visual>
-        <!-- <collision> -->
-            <!-- <origin xyz="0 0 0" rpy="0 0 0"/> -->
-            <!-- <geometry> -->
-                <!-- <box size="0.4 0.3 0.01"/> -->
-            <!-- </geometry> -->
-        <!-- </collision> -->
+        <collision>
+            <origin xyz="0 0 0" rpy="0 0 0"/>
+            <geometry>
+                <box size="0.4 0.3 0.01"/>
+            </geometry>
+        </collision>
     </link>
     <joint name="front_plate_joint" type="fixed">
@@ -167,10 +189,10 @@
             <material name="silver"/>
         </visual>
-        <!-- <collision> -->
-            <!-- <origin xyz="0 0 0" rpy="0 0 0"/> -->
-            <!-- <geometry> -->
-                <!-- <box size="0.4 0.3 0.01"/> -->
-            <!-- </geometry> -->
-        <!-- </collision> -->
+        <collision>
+            <origin xyz="0 0 0" rpy="0 0 0"/>
+            <geometry>
+                <box size="0.4 0.3 0.01"/>
+            </geometry>
+        </collision>
     </link>
     <joint name="rear_plate_joint" type="fixed">
@@ -190,10 +212,10 @@
             <material name="black"/>
         </visual>
-        <!-- <collision> -->
-            <!-- <origin xyz="0 0 0" rpy="0 0 0"/> -->
-            <!-- <geometry> -->
-                <!-- <box size="0.12 0.01 0.01"/> -->
-            <!-- </geometry> -->
-        <!-- </collision> -->
+        <collision>
+            <origin xyz="0 0 0" rpy="0 0 0"/>
+            <geometry>
+                <box size="0.12 0.01 0.01"/>
+            </geometry>
+        </collision>
     </link>
     <joint name="rear_trans_chassis_joint" type="fixed">
@@ -213,10 +235,10 @@
             <material name="black"/>
         </visual>
-        <!-- <collision> -->
-            <!-- <origin xyz="0 0 0" rpy="0 0 0"/> -->
-            <!-- <geometry> -->
-                <!-- <cylinder radius="0.02" length="0.28"/> -->
-            <!-- </geometry> -->
-        <!-- </collision> -->
+        <collision>
+            <origin xyz="0 0 0" rpy="0 0 0"/>
+            <geometry>
+                <cylinder radius="0.02" length="0.28"/>
+            </geometry>
+        </collision>
     </link>
     <joint name="rear_trans_joint" type="fixed">
@@ -238,10 +260,10 @@
             </material>
         </visual>
-        <!-- <collision> -->
-            <!-- <origin xyz="0 0 0" rpy="0 0 0"/> -->
-            <!-- <geometry> -->
-                <!-- <mesh filename="package://kymco_maxxer90_description/meshes/spring.stl" scale="1.0 1.0 1.0"/> -->
-            <!-- </geometry> -->
-        <!-- </collision> -->
+        <collision>
+            <origin xyz="0 0 0" rpy="0 0 0"/>
+            <geometry>
+                <mesh filename="package://kymco_maxxer90_description/meshes/spring.stl" scale="1.0 1.0 1.0"/>
+            </geometry>
+        </collision>
     </link>
     <gazebo reference="rear_trans_spring_link">
@@ -261,10 +283,10 @@
             <material name="black"/>
         </visual>
-        <!-- <collision> -->
-            <!-- <origin xyz="0 0 0" rpy="0 0 0"/> -->
-            <!-- <geometry> -->
-                <!-- <box size="0.01 0.2 0.01"/> -->
-            <!-- </geometry> -->
-        <!-- </collision> -->
+        <collision>
+            <origin xyz="0 0 0" rpy="0 0 0"/>
+            <geometry>
+                <box size="0.01 0.2 0.01"/>
+            </geometry>
+        </collision>
     </link>
     <joint name="front_right_trans_chassis_joint" type="fixed">
@@ -284,10 +306,10 @@
             <material name="black"/>
         </visual>
-        <!-- <collision> -->
-            <!-- <origin xyz="0 0 0" rpy="0 0 0"/> -->
-            <!-- <geometry> -->
-                <!-- <cylinder radius="0.02" length="0.28"/> -->
-            <!-- </geometry> -->
-        <!-- </collision> -->
+        <collision>
+            <origin xyz="0 0 0" rpy="0 0 0"/>
+            <geometry>
+                <cylinder radius="0.02" length="0.28"/>
+            </geometry>
+        </collision>
     </link>
     <joint name="front_right_trans_joint" type="fixed">
@@ -309,10 +331,10 @@
             </material>
         </visual>
-        <!-- <collision> -->
-            <!-- <origin xyz="0 0 0" rpy="0 0 0"/> -->
-            <!-- <geometry> -->
-                <!-- <mesh filename="package://kymco_maxxer90_description/meshes/spring.stl" scale="1.0 1.0 1.0"/> -->
-            <!-- </geometry> -->
-        <!-- </collision> -->
+        <collision>
+            <origin xyz="0 0 0" rpy="0 0 0"/>
+            <geometry>
+                <mesh filename="package://kymco_maxxer90_description/meshes/spring.stl" scale="1.0 1.0 1.0"/>
+            </geometry>
+        </collision>
     </link>
     <joint name="front_right_trans_spring_joint" type="fixed">
@@ -332,10 +354,10 @@
             <material name="black"/>
         </visual>
-        <!-- <collision> -->
-            <!-- <origin xyz="0 0 0" rpy="0 0 0"/> -->
-            <!-- <geometry> -->
-                <!-- <box size="0.01 0.2 0.01"/> -->
-            <!-- </geometry> -->
-        <!-- </collision> -->
+        <collision>
+            <origin xyz="0 0 0" rpy="0 0 0"/>
+            <geometry>
+                <box size="0.01 0.2 0.01"/>
+            </geometry>
+        </collision>
     </link>
     <joint name="front_left_trans_chassis_joint" type="fixed">
@@ -355,10 +377,10 @@
             <material name="black"/>
         </visual>
-        <!-- <collision> -->
-            <!-- <origin xyz="0 0 0" rpy="0 0 0"/> -->
-            <!-- <geometry> -->
-                <!-- <cylinder radius="0.02" length="0.28"/> -->
-            <!-- </geometry> -->
-        <!-- </collision> -->
+        <collision>
+            <origin xyz="0 0 0" rpy="0 0 0"/>
+            <geometry>
+                <cylinder radius="0.02" length="0.28"/>
+            </geometry>
+        </collision>
     </link>
     <joint name="front_left_trans_joint" type="fixed">
@@ -380,10 +402,10 @@
             </material>
         </visual>
-        <!-- <collision> -->
-            <!-- <origin xyz="0 0 0" rpy="0 0 0"/> -->
-            <!-- <geometry> -->
-                <!-- <mesh filename="package://kymco_maxxer90_description/meshes/spring.stl" scale="1.0 1.0 1.0"/> -->
-            <!-- </geometry> -->
-        <!-- </collision> -->
+        <collision>
+            <origin xyz="0 0 0" rpy="0 0 0"/>
+            <geometry>
+                <mesh filename="package://kymco_maxxer90_description/meshes/spring.stl" scale="1.0 1.0 1.0"/>
+            </geometry>
+        </collision>
     </link>
     <joint name="front_left_trans_spring_joint" type="fixed">
@@ -395,3 +417,11 @@
         <material>Gazebo/Red</material>
     </gazebo>"
+    <gazebo>
+      <plugin name="ros_control" filename="libgazebo_ros_control.so">
+        <robotNamespace></robotNamespace>
+        <robotParam>robot_description</robotParam>
+        <controlPeriod>0.001</controlPeriod>
+	    <robotSimType>gazebo_ros_control/DefaultRobotHWSim</robotSimType>
+      </plugin>
+    </gazebo>
 </robot>

File: kymco_maxxer90_description/urdf/wheel.urdf.xacro (robot description, xacro)
@@ -23,5 +23,5 @@
 		</link>
 		<joint name="${wheel_prefix}_wheel" type="continuous">
-			<parent link="base_link"/>
+			<parent link="RWD"/>
 			<child link="${wheel_prefix}_wheel_link"/>
 			<xacro:insert_block name="joint_pose"/>
@@ -37,5 +37,5 @@
             </actuator>
             <joint name="${wheel_prefix}_wheel">
-                <hardwareInterface>VelocityJointInterface</hardwareInterface>
+                <hardwareInterface>hardware_interface/VelocityJointInterface</hardwareInterface>
             </joint>
         </transmission>

Commit message: First working version without suspension

File: kymco_maxxer90_description/urdf/front_wheel.urdf.xacro (robot description, xacro)
@@ -37,5 +37,5 @@
             <!-- TODO effort and velocity -->
             <limit lower="${-PI*25/180}" upper="${PI*25/180}" effort="100.5" velocity="4.5"/>
-            <dynamics damping="0.2" friction="0" />
+            <dynamics damping="3" friction="0.0" />
         </joint>
 		<joint name="${wheel_prefix}_wheel" type="continuous">
@@ -55,6 +55,6 @@
                 <multiplier>1.0</multiplier>
                 <offset>0</offset>
-                <sensitiveness>0.0</sensitiveness>
-                <maxEffort>10.0</maxEffort>
+                <sensitiveness>0.1</sensitiveness>
+                <maxEffort>100000.0</maxEffort>
             </plugin>
         </gazebo>

File: kymco_maxxer90_description/urdf/kymco_maxxer90.urdf.xacro (robot description, xacro)
@@ -63,5 +63,5 @@
         <!-- TODO effort and velocity -->
         <limit lower="${-PI*25/180}" upper="${PI*25/180}" effort="100.5" velocity="4.5"/>
-        <dynamics damping="20" friction="2.0" />
+        <dynamics damping="3" friction="0.0" />
     </joint>
     <transmission name="steering_wheel_joint_trans">
@@ -138,5 +138,5 @@
     <link name="RWD">
         <inertial>
-            <mass value="1"/>
+            <mass value="5"/>
             <origin xyz="0 0 0"/>
             <inertia ixx="0.01" ixy="0" ixz="0" iyy="0.01" iyz="0" izz="0.01"/>

Commit message: Added front suspension. I need to tweak stifness and play with inertia

File: kymco_maxxer90_description/urdf/front_wheel.urdf.xacro (robot description, xacro)
@@ -29,7 +29,28 @@
             </inertial>
         </link>
+        <link name="${wheel_prefix}_suspension_link" >
+            <inertial>
+                <mass value="1"/>
+                <origin xyz="0 0 0"/>
+                <inertia ixx="0.01" ixy="0" ixz="0" iyy="0.01" iyz="0" izz="0.01"/>
+            </inertial>
+        </link>
+        <joint name="${wheel_prefix}_suspension_joint" type="prismatic">
+			<xacro:insert_block name="joint_pose"/>
+            <parent link="base_link"/>
+            <child link="${wheel_prefix}_suspension_link"/>
+            <axis xyz="0 0 -1" />
+            <limit lower="-0.1" upper="0.1" effort="500" velocity="10"/>
+            <!-- <dynamics damping="1" friction="0.2"/> -->
+        </joint>
+        <gazebo reference="${wheel_prefix}_suspension_joint">
+            <provideFeedback>true</provideFeedback>
+            <implicitSpringDamper>true</implicitSpringDamper>
+            <springStiffness>30000</springStiffness>
+            <springReference>0</springReference>
+        </gazebo>
         <joint name="${wheel_prefix}_steering_wheel_joint" type="revolute">
-			<xacro:insert_block name="joint_pose"/>
-			<parent link="base_link"/>
+            <origin xyz="0 0 0" rpy="0 0 0" />
+            <parent link="${wheel_prefix}_suspension_link"/>
 			<child link="${wheel_prefix}_wheel_steering_link"/>
             <axis xyz="0 0 1" />

Commit message: Fixed steering after the addition of suspension on the front, and also fixed joint state publishing by adding transmission to some joints

File: kymco_maxxer90_description/urdf/front_wheel.urdf.xacro (robot description, xacro)
@@ -50,4 +50,13 @@
             <springReference>0</springReference>
         </gazebo>
+        <transmission name="${wheel_prefix}_suspension_trans" type="SimpleTransmission">
+        <type>transmission_interface/SimpleTransmission</type>
+        <actuator name="${wheel_prefix}_suspension_actuator">
+            <mechanicalReduction>1</mechanicalReduction>
+        </actuator>
+        <joint name="${wheel_prefix}_suspension_joint">
+            <hardwareInterface>hardware_interface/EffortJointInterface</hardwareInterface>
+        </joint>
+    </transmission>
         <joint name="${wheel_prefix}_steering_wheel_joint" type="revolute">
             <origin xyz="0 0 0" rpy="0 0 0" />
@@ -69,4 +78,13 @@
             <material>Gazebo/Black</material>
         </gazebo>"
+        <transmission name="${wheel_prefix}_wheel_trans" type="SimpleTransmission">
+        <type>transmission_interface/SimpleTransmission</type>
+        <actuator name="${wheel_prefix}_wheel_actuator">
+            <mechanicalReduction>0</mechanicalReduction>
+        </actuator>
+        <joint name="${wheel_prefix}_wheel">
+            <hardwareInterface>hardware_interface/EffortJointInterface</hardwareInterface>
+        </joint>
+    </transmission>
         <gazebo>
             <plugin name="${wheel_prefix}_mimic_joint_plugin" filename="libroboticsgroup_gazebo_mimic_joint_plugin.so">
@@ -80,22 +98,4 @@
             </plugin>
         </gazebo>
-        <!-- <transmission name="${wheel_prefix}_wheel_steering_joint_trans"> -->
-            <!-- <type>transmission_interface/SimpleTransmission</type> -->
-            <!-- <joint name="${wheel_prefix}_steering_wheel_joint"> -->
-                <!-- <hardwareInterface>hardware_interface/PositionJointInterface</hardwareInterface> -->
-            <!-- </joint> -->
-            <!-- <actuator name="${wheel_prefix}_steering_wheel_actuator"> -->
-                <!-- <mechanicalReduction>1</mechanicalReduction> -->
-            <!-- </actuator> -->
-        <!-- </transmission> -->
-        <!-- <transmission name="${wheel_prefix}_wheel_trans" type="SimpleTransmission"> -->
-            <!-- <type>transmission_interface/SimpleTransmission</type> -->
-            <!-- <actuator name="${wheel_prefix}_wheel_motor"> -->
-                <!-- <mechanicalReduction>0</mechanicalReduction> -->
-            <!-- </actuator> -->
-            <!-- <joint name="${wheel_prefix}_wheel"> -->
-                <!-- <hardwareInterface>hardware_interface/VelocityJointInterface</hardwareInterface> -->
-            <!-- </joint> -->
-        <!-- </transmission> -->
 	</xacro:macro>
 </robot>

File: kymco_maxxer90_description/urdf/kymco_maxxer90.urdf.xacro (robot description, xacro)
@@ -134,4 +134,13 @@
         <springReference>0</springReference>
     </gazebo>
+    <transmission name="rear_suspension_trans" type="SimpleTransmission">
+        <type>transmission_interface/SimpleTransmission</type>
+        <actuator name="rear_suspension_actuator">
+            <mechanicalReduction>1</mechanicalReduction>
+        </actuator>
+        <joint name="rear_suspension_joint">
+            <hardwareInterface>hardware_interface/EffortJointInterface</hardwareInterface>
+        </joint>
+    </transmission>
     <link name="rear_axle_link">
         <visual>
