Commit message: Sanitizing inertia but still not working on Gazebo 9 (it does on Gazebo11)

File: kymco_maxxer90_description/urdf/front_wheel.urdf.xacro (robot description, xacro)
@@ -24,7 +24,7 @@
         <link name="${wheel_prefix}_wheel_steering_link" >
             <inertial>
-                <mass value="1"/>
+                <mass value="0.01"/>
                 <origin xyz="0 0 0"/>
-                <inertia ixx="0.01" ixy="0" ixz="0" iyy="0.01" iyz="0" izz="0.01"/>
+                <inertia ixx="0.0001" ixy="0" ixz="0" iyy="0.0001" iyz="0" izz="0.0001"/>
             </inertial>
         </link>
@@ -44,19 +44,19 @@
             <!-- <dynamics damping="1" friction="0.2"/> -->
         </joint>
-        <gazebo reference="${wheel_prefix}_suspension_joint">
-            <provideFeedback>true</provideFeedback>
-            <implicitSpringDamper>true</implicitSpringDamper>
-            <springStiffness>30000</springStiffness>
-            <springReference>0</springReference>
-        </gazebo>
+        <!-- <gazebo reference="${wheel_prefix}_suspension_joint"> -->
+            <!-- <provideFeedback>true</provideFeedback> -->
+            <!-- <implicitSpringDamper>true</implicitSpringDamper> -->
+            <!-- <springStiffness>30000</springStiffness> -->
+            <!-- <springReference>0</springReference> -->
+        <!-- </gazebo> -->
         <transmission name="${wheel_prefix}_suspension_trans" type="SimpleTransmission">
-        <type>transmission_interface/SimpleTransmission</type>
-        <actuator name="${wheel_prefix}_suspension_actuator">
-            <mechanicalReduction>1</mechanicalReduction>
-        </actuator>
-        <joint name="${wheel_prefix}_suspension_joint">
-            <hardwareInterface>hardware_interface/EffortJointInterface</hardwareInterface>
-        </joint>
-    </transmission>
+            <type>transmission_interface/SimpleTransmission</type>
+            <actuator name="${wheel_prefix}_suspension_actuator">
+                <mechanicalReduction>1</mechanicalReduction>
+            </actuator>
+            <joint name="${wheel_prefix}_suspension_joint">
+                <hardwareInterface>hardware_interface/EffortJointInterface</hardwareInterface>
+            </joint>
+        </transmission>
         <joint name="${wheel_prefix}_steering_wheel_joint" type="revolute">
             <origin xyz="0 0 0" rpy="0 0 0" />
@@ -66,6 +66,6 @@
             <mimic joint="steering_wheel_joint" multiplier="1" offset="0" />
             <!-- TODO effort and velocity -->
-            <limit lower="${-PI*25/180}" upper="${PI*25/180}" effort="100.5" velocity="4.5"/>
-            <dynamics damping="3" friction="0.0" />
+            <limit lower="${-PI*25/180}" upper="${PI*25/180}" effort="100000" velocity="0.95"/>
+            <dynamics damping="0" friction="0.0" />
         </joint>
 		<joint name="${wheel_prefix}_wheel" type="continuous">
@@ -79,12 +79,12 @@
         </gazebo>"
         <transmission name="${wheel_prefix}_wheel_trans" type="SimpleTransmission">
-        <type>transmission_interface/SimpleTransmission</type>
-        <actuator name="${wheel_prefix}_wheel_actuator">
-            <mechanicalReduction>0</mechanicalReduction>
-        </actuator>
-        <joint name="${wheel_prefix}_wheel">
-            <hardwareInterface>hardware_interface/EffortJointInterface</hardwareInterface>
-        </joint>
-    </transmission>
+            <type>transmission_interface/SimpleTransmission</type>
+            <actuator name="${wheel_prefix}_wheel_actuator">
+                <mechanicalReduction>0</mechanicalReduction>
+            </actuator>
+            <joint name="${wheel_prefix}_wheel">
+                <hardwareInterface>hardware_interface/EffortJointInterface</hardwareInterface>
+            </joint>
+        </transmission>
         <gazebo>
             <plugin name="${wheel_prefix}_mimic_joint_plugin" filename="libroboticsgroup_gazebo_mimic_joint_plugin.so">
@@ -94,6 +94,6 @@
                 <multiplier>1.0</multiplier>
                 <offset>0</offset>
-                <sensitiveness>0.1</sensitiveness>
-                <maxEffort>100000.0</maxEffort>
+                <sensitiveness>0.0</sensitiveness>
+                <maxEffort>1000000.0</maxEffort>
             </plugin>
         </gazebo>

Commit message: Now steering properly in Gazebo9 too

File: kymco_maxxer90_description/urdf/front_wheel.urdf.xacro (robot description, xacro)
@@ -42,12 +42,11 @@
             <axis xyz="0 0 -1" />
             <limit lower="-0.1" upper="0.1" effort="500" velocity="10"/>
-            <!-- <dynamics damping="1" friction="0.2"/> -->
         </joint>
-        <!-- <gazebo reference="${wheel_prefix}_suspension_joint"> -->
-            <!-- <provideFeedback>true</provideFeedback> -->
-            <!-- <implicitSpringDamper>true</implicitSpringDamper> -->
-            <!-- <springStiffness>30000</springStiffness> -->
-            <!-- <springReference>0</springReference> -->
-        <!-- </gazebo> -->
+        <gazebo reference="${wheel_prefix}_suspension_joint">
+            <provideFeedback>true</provideFeedback>
+            <implicitSpringDamper>true</implicitSpringDamper>
+            <springStiffness>30000</springStiffness>
+            <springReference>0</springReference>
+        </gazebo>
         <transmission name="${wheel_prefix}_suspension_trans" type="SimpleTransmission">
             <type>transmission_interface/SimpleTransmission</type>
@@ -67,5 +66,5 @@
             <!-- TODO effort and velocity -->
             <limit lower="${-PI*25/180}" upper="${PI*25/180}" effort="100000" velocity="0.95"/>
-            <dynamics damping="0" friction="0.0" />
+            <dynamics damping="0" friction="1.0" />
         </joint>
 		<joint name="${wheel_prefix}_wheel" type="continuous">

Commit message: Added gps and imu on simulation. Still fighting with inertia

File: kymco_maxxer90_description/urdf/front_wheel.urdf.xacro (robot description, xacro)
@@ -4,7 +4,7 @@
 		<link name="${wheel_prefix}_wheel_link">
             <inertial>
-                <mass value="15.0"/>
+                <mass value="8.0"/>
                 <origin xyz="0 0 0"/>
-                <inertia  ixx="0.28813432952881635" ixy="0" ixz="0" iyy="0.5212991167201597" iyz="0" izz="0.2894147916616918" />
+                <inertia  ixx="0.11952" ixy="0" ixz="0" iyy="0.20903" iyz="0" izz="0.11952" />
             </inertial>
 			<visual>
@@ -16,7 +16,9 @@
 			</visual>
 			<collision>
-                <origin xyz="0 0 0" rpy="0 0 0" />
+                <!-- <origin xyz="0 0 0" rpy="0 0 0" /> -->
+                <origin xyz="0 0 0" rpy="${PI/2} 0 0" />
 				<geometry>
-                    <mesh filename="package://kymco_maxxer90_description/meshes/wheel.stl" scale="1.0 1.0 1.0"/>
+                    <!-- <mesh filename="package://kymco_maxxer90_description/meshes/wheel.stl" scale="1.0 1.0 1.0"/> -->
+                    <cylinder radius="0.2286" length="0.15" />
 				</geometry>
 			</collision>
@@ -24,5 +26,5 @@
         <link name="${wheel_prefix}_wheel_steering_link" >
             <inertial>
-                <mass value="0.01"/>
+                <mass value="1"/>
                 <origin xyz="0 0 0"/>
                 <inertia ixx="0.0001" ixy="0" ixz="0" iyy="0.0001" iyz="0" izz="0.0001"/>
@@ -33,5 +35,5 @@
                 <mass value="1"/>
                 <origin xyz="0 0 0"/>
-                <inertia ixx="0.01" ixy="0" ixz="0" iyy="0.01" iyz="0" izz="0.01"/>
+                <inertia ixx="0.005" ixy="0" ixz="0" iyy="0.005" iyz="0" izz="0.005"/>
             </inertial>
         </link>
@@ -64,5 +66,4 @@
             <axis xyz="0 0 1" />
             <mimic joint="steering_wheel_joint" multiplier="1" offset="0" />
-            <!-- TODO effort and velocity -->
             <limit lower="${-PI*25/180}" upper="${PI*25/180}" effort="100000" velocity="0.95"/>
             <dynamics damping="0" friction="1.0" />

File: kymco_maxxer90_description/urdf/kymco_maxxer90.urdf.xacro (robot description, xacro)
@@ -51,5 +51,5 @@
     <link name="steering_wheel_link">
         <inertial>
-            <mass value="0.01"/>
+            <mass value="20"/>
             <origin xyz="0 0 0"/>
             <inertia ixx="0.0001" ixy="0" ixz="0" iyy="0.0001" iyz="0" izz="0.0001"/>
@@ -61,5 +61,4 @@
         <child link="steering_wheel_link" />
         <axis xyz="0 0 1" />
-        <!-- TODO effort and velocity -->
         <limit lower="${-PI*25/180}" upper="${PI*25/180}" effort="100000" velocity="0.95"/>
         <dynamics damping="0" friction="0.0" />
@@ -115,7 +114,7 @@
     <link name="rear_suspension_link" >
         <inertial>
-            <mass value="1"/>
+            <mass value="10"/>
             <origin xyz="0 0 0"/>
-            <inertia ixx="0.01" ixy="0" ixz="0" iyy="0.01" iyz="0" izz="0.01"/>
+            <inertia ixx="0.005" ixy="0" ixz="0" iyy="0.005" iyz="0" izz="0.005"/>
         </inertial>
     </link>
@@ -168,7 +167,7 @@
     <link name="RWD">
         <inertial>
-            <mass value="1"/>
+            <mass value="10"/>
             <origin xyz="0 0 0"/>
-            <inertia ixx="0.01" ixy="0" ixz="0" iyy="0.01" iyz="0" izz="0.01"/>
+            <inertia ixx="0.005" ixy="0" ixz="0" iyy="0.005" iyz="0" izz="0.005"/>
         </inertial>
     </link>
@@ -447,11 +446,48 @@
         <material>Gazebo/Red</material>
     </gazebo>"
+    <!-- Sensors -->
+    <link name="gps_link"/>
+    <joint name="gps_joint" type="fixed">
+        <origin xyz="0 0 0" rpy="0 0 0"/>
+        <parent link="base_link" />
+        <child link="gps_link" />
+    </joint>
+    <link name="imu_link"/>
+    <joint name="imu_joint" type="fixed">
+        <origin xyz="0 0 0" rpy="0 0 0"/>
+        <parent link="base_link"/>
+        <child link="imu_link"/>
+    </joint>
+    <!-- Gazebo plugins -->
     <gazebo>
-      <plugin name="ros_control" filename="libgazebo_ros_control.so">
-        <robotNamespace></robotNamespace>
-        <robotParam>robot_description</robotParam>
-        <controlPeriod>0.001</controlPeriod>
-	    <robotSimType>gazebo_ros_control/DefaultRobotHWSim</robotSimType>
-      </plugin>
+        <plugin name="gps_controller" filename="libhector_gazebo_ros_gps.so">
+            <robotNamespace>/</robotNamespace>
+            <updateRate>40</updateRate>
+            <bodyName>base_link</bodyName>
+            <frameId>base_link</frameId>
+            <topicName>navsat/fix</topicName>
+            <velocityTopicName>navsat/vel</velocityTopicName>
+            <referenceLatitude>37.9949</referenceLatitude>
+            <referenceLongitude>23.819173</referenceLongitude>
+            <referenceHeading>0</referenceHeading>
+            <referenceAltitude>0</referenceAltitude>
+            <drift>0.0001 0.0001 0.0001</drift>
+        </plugin>
+        <plugin name="jaguar_imu_sensor" filename="libhector_gazebo_ros_imu.so">
+            <updateRate>50.0</updateRate>
+            <bodyName>base_link</bodyName>
+            <frameId>base_link</frameId>
+            <topicName>imu/data</topicName>
+            <accelDrift>0.00001 0.00001 0.00001</accelDrift>
+            <accelGaussianNoise>0.001 0.001 0.001</accelGaussianNoise>
+            <rateDrift>0.001 0.001 0.001</rateDrift>
+            <rateGaussianNoise>0.01 0.01 0.01</rateGaussianNoise>
+        </plugin>
+        <plugin name="ros_control" filename="libgazebo_ros_control.so">
+            <robotNamespace></robotNamespace>
+            <robotParam>robot_description</robotParam>
+            <controlPeriod>0.001</controlPeriod>
+            <robotSimType>gazebo_ros_control/DefaultRobotHWSim</robotSimType>
+        </plugin>
     </gazebo>
 </robot>

File: kymco_maxxer90_description/urdf/wheel.urdf.xacro (robot description, xacro)
@@ -4,10 +4,10 @@
 		<link name="${wheel_prefix}_wheel_link">
 			<inertial>
-				<mass value="15.0" />
+				<mass value="10.0" />
                 <origin xyz="0 0 0" />
-                <inertia  ixx="0.28813432952881635" ixy="0" ixz="0" iyy="0.5212991167201597" iyz="0" izz="0.2894147916616918" />
+                <inertia  ixx="0.1494" ixy="0" ixz="0" iyy="0.2613" iyz="0" izz="0.1494" />
 			</inertial>
 			<visual>
-				<origin xyz="0 0 0" rpy="0 0 0" />
+                <origin xyz="0 0 0" rpy="0 0 0" />
 				<geometry>
                     <mesh filename="package://kymco_maxxer90_description/meshes/wheel.stl" scale="1.0 1.0 1.0"/>
@@ -16,7 +16,9 @@
 			</visual>
 			<collision>
-                <origin xyz="0 0 0" rpy="0 0 0" />
+                <!-- <origin xyz="0 0 0" rpy="0 0 0" /> -->
+                <origin xyz="0 0 0" rpy="${PI/2} 0 0" />
 				<geometry>
-                    <mesh filename="package://kymco_maxxer90_description/meshes/wheel.stl" scale="1.0 1.0 1.0"/>
+                    <!-- <mesh filename="package://kymco_maxxer90_description/meshes/wheel.stl" scale="1.0 1.0 1.0"/> -->
+                    <cylinder radius="0.2286" length="0.15" />
 				</geometry>
 			</collision>

Commit message: Improved robot overall oscillation

File: kymco_maxxer90_description/urdf/front_wheel.urdf.xacro (robot description, xacro)
@@ -74,4 +74,5 @@
 			<child link="${wheel_prefix}_wheel_link"/>
 			<axis xyz="0 1 0" rpy="0 0 0" />
+            <dynamics damping="0.1" friction="0.1" />
         </joint>
         <gazebo reference="${wheel_prefix}_wheel_link">

File: kymco_maxxer90_description/urdf/kymco_maxxer90.urdf.xacro (robot description, xacro)
@@ -44,16 +44,16 @@
     <link name="steering_wheel_link">
         <inertial>
-            <mass value="2"/>
+            <mass value="5"/>
             <origin xyz="0 0 0"/>
-            <inertia ixx="0.0001" ixy="0" ixz="0" iyy="0.0001" iyz="0" izz="0.0001"/>
+            <inertia ixx="0.01" ixy="0" ixz="0" iyy="0.01" iyz="0" izz="0.01"/>
         </inertial>
     </link>
     <joint name="steering_wheel_joint" type="revolute">
-        <origin xyz="0 0 0" rpy="0 0 0" />
+        <origin xyz="-0.3 0 0.8" rpy="0 0 0" />
         <parent link="base_link" />
         <child link="steering_wheel_link" />
         <axis xyz="0 0 1" />
         <limit lower="${-PI*25/180}" upper="${PI*25/180}" effort="100000" velocity="0.95"/>
-        <dynamics damping="0" friction="0.0" />
+        <dynamics damping="10" friction="0.3" />
     </joint>
     <transmission name="steering_wheel_joint_trans">

File: kymco_maxxer90_description/urdf/wheel.urdf.xacro (robot description, xacro)
@@ -29,4 +29,5 @@
 			<xacro:insert_block name="joint_pose"/>
 			<axis xyz="0 1 0" rpy="0 0 0" />
+            <dynamics damping="1" friction="1" />
 		</joint>
         <gazebo reference="${wheel_prefix}_wheel_link">
