Commit message: More additions towards a realistic robot description

File: kymco_maxxer90_description/urdf/kymco_maxxer90.urdf.xacro (robot description, xacro)
@@ -75,5 +75,5 @@
     </link>
     <joint name="rear_axle_joint" type="fixed">
-        <origin xyz="0.03 ${0.33-wheelbase} ${distance_from_ground-wheel_diameter/2}" rpy="0 0 ${-PI/2}"/>
+        <origin xyz="0.03 ${0.33-wheelbase} ${distance_from_ground/2}" rpy="0 0 ${-PI/2}"/>
         <parent link="base_link" />
         <child link="rear_axle_link" />
@@ -95,5 +95,5 @@
     </link>
     <joint name="front_plate_joint" type="fixed">
-        <origin xyz="0 0.45 0.56" rpy="0 0 0"/>
+        <origin xyz="0 0.45 0.561" rpy="0 0 0"/>
         <parent link="base_link" />
         <child link="front_plate_link" />
@@ -119,3 +119,209 @@
         <child link="rear_plate_link" />
     </joint>
+    <link name="rear_trans_chassis_link">
+        <visual>
+            <origin xyz="0 0 0" rpy="0 0 0"/>
+            <geometry>
+                <box size="0.12 0.01 0.01"/>
+            </geometry>
+            <material name="black"/>
+        </visual>
+        <collision>
+            <origin xyz="0 0 0" rpy="0 0 0"/>
+            <geometry>
+                <box size="0.12 0.01 0.01"/>
+            </geometry>
+        </collision>
+    </link>
+    <joint name="rear_trans_chassis_joint" type="fixed">
+        <origin xyz="0 -0.46 0.39" rpy="0 0 0"/>
+        <parent link="base_link" />
+        <child link="rear_trans_chassis_link" />
+    </joint>
+    <link name="rear_trans_link">
+        <visual>
+            <origin xyz="0 0 0" rpy="0 0 0"/>
+            <geometry>
+                <cylinder radius="0.02" length="0.28"/>
+            </geometry>
+            <material name="black"/>
+        </visual>
+        <collision>
+            <origin xyz="0 0 0" rpy="0 0 0"/>
+            <geometry>
+                <cylinder radius="0.02" length="0.28"/>
+            </geometry>
+        </collision>
+    </link>
+    <joint name="rear_trans_joint" type="fixed">
+        <origin xyz="0 -0.56 0.29" rpy="${-PI/4} 0 0"/>
+        <parent link="base_link" />
+        <child link="rear_trans_link" />
+    </joint>
+    <link name="rear_trans_spring_link">
+        <visual>
+            <origin xyz="0 0 0" rpy="0 0 0"/>
+            <geometry>
+                <mesh filename="package://kymco_maxxer90_description/meshes/spring.stl" scale="1.0 1.0 1.0"/>
+            </geometry>
+            <material name="red">
+                <color rgba="0.8 0 0 1"/>
+            </material>
+        </visual>
+        <collision>
+            <origin xyz="0 0 0" rpy="0 0 0"/>
+            <geometry>
+                <mesh filename="package://kymco_maxxer90_description/meshes/spring.stl" scale="1.0 1.0 1.0"/>
+            </geometry>
+        </collision>
+    </link>
+    <joint name="rear_trans_spring_joint" type="fixed">
+        <origin xyz="0 -0.56 0.29" rpy="${-PI/4} 0 0"/>
+        <parent link="base_link" />
+        <child link="rear_trans_spring_link" />
+    </joint>
+    <link name="front_right_trans_chassis_link">
+        <visual>
+            <origin xyz="0 0 0" rpy="0 0 0"/>
+            <geometry>
+                <box size="0.01 0.2 0.01"/>
+            </geometry>
+            <material name="black"/>
+        </visual>
+        <collision>
+            <origin xyz="0 0 0" rpy="0 0 0"/>
+            <geometry>
+                <box size="0.01 0.2 0.01"/>
+            </geometry>
+        </collision>
+    </link>
+    <joint name="front_right_trans_chassis_joint" type="fixed">
+        <origin xyz="0.075 0.33 0.4" rpy="0 0 0"/>
+        <parent link="base_link" />
+        <child link="front_right_trans_chassis_link" />
+    </joint>
+    <link name="front_right_trans_link">
+        <visual>
+            <origin xyz="0 0 0" rpy="0 0 0"/>
+            <geometry>
+                <cylinder radius="0.02" length="0.28"/>
+            </geometry>
+            <material name="black"/>
+        </visual>
+        <collision>
+            <origin xyz="0 0 0" rpy="0 0 0"/>
+            <geometry>
+                <cylinder radius="0.02" length="0.28"/>
+            </geometry>
+        </collision>
+    </link>
+    <joint name="front_right_trans_joint" type="fixed">
+        <origin xyz="0.15 0.33 0.29" rpy="${PI/10} ${-PI/5} 0"/>
+        <parent link="base_link" />
+        <child link="front_right_trans_link" />
+    </joint>
+    <link name="front_right_trans_spring_link">
+        <visual>
+            <origin xyz="0 0 0" rpy="0 0 0"/>
+            <geometry>
+                <mesh filename="package://kymco_maxxer90_description/meshes/spring.stl" scale="1.0 1.0 1.0"/>
+            </geometry>
+            <material name="red">
+                <color rgba="0.8 0 0 1"/>
+            </material>
+        </visual>
+        <collision>
+            <origin xyz="0 0 0" rpy="0 0 0"/>
+            <geometry>
+                <mesh filename="package://kymco_maxxer90_description/meshes/spring.stl" scale="1.0 1.0 1.0"/>
+            </geometry>
+        </collision>
+    </link>
+    <joint name="front_right_trans_spring_joint" type="fixed">
+        <origin xyz="0.15 0.33 0.29" rpy="${PI/10} ${-PI/5} 0"/>
+        <parent link="base_link" />
+        <child link="front_right_trans_spring_link" />
+    </joint>
+    <link name="front_left_trans_chassis_link">
+        <visual>
+            <origin xyz="0 0 0" rpy="0 0 0"/>
+            <geometry>
+                <box size="0.01 0.2 0.01"/>
+            </geometry>
+            <material name="black"/>
+        </visual>
+        <collision>
+            <origin xyz="0 0 0" rpy="0 0 0"/>
+            <geometry>
+                <box size="0.01 0.2 0.01"/>
+            </geometry>
+        </collision>
+    </link>
+    <joint name="front_left_trans_chassis_joint" type="fixed">
+        <origin xyz="-0.075 0.33 0.4" rpy="0 0 0"/>
+        <parent link="base_link" />
+        <child link="front_left_trans_chassis_link" />
+    </joint>
+    <link name="front_left_trans_link">
+        <visual>
+            <origin xyz="0 0 0" rpy="0 0 0"/>
+            <geometry>
+                <cylinder radius="0.02" length="0.28"/>
+            </geometry>
+            <material name="black"/>
+        </visual>
+        <collision>
+            <origin xyz="0 0 0" rpy="0 0 0"/>
+            <geometry>
+                <cylinder radius="0.02" length="0.28"/>
+            </geometry>
+        </collision>
+    </link>
+    <joint name="front_left_trans_joint" type="fixed">
+        <origin xyz="-0.15 0.33 0.29" rpy="${PI/10} ${PI/5} 0"/>
+        <parent link="base_link" />
+        <child link="front_left_trans_link" />
+    </joint>
+    <link name="front_left_trans_spring_link">
+        <visual>
+            <origin xyz="0 0 0" rpy="0 0 0"/>
+            <geometry>
+                <mesh filename="package://kymco_maxxer90_description/meshes/spring.stl" scale="1.0 1.0 1.0"/>
+            </geometry>
+            <material name="red">
+                <color rgba="0.8 0 0 1"/>
+            </material>
+        </visual>
+        <collision>
+            <origin xyz="0 0 0" rpy="0 0 0"/>
+            <geometry>
+                <mesh filename="package://kymco_maxxer90_description/meshes/spring.stl" scale="1.0 1.0 1.0"/>
+            </geometry>
+        </collision>
+    </link>
+    <joint name="front_left_trans_spring_joint" type="fixed">
+        <origin xyz="-0.15 0.33 0.29" rpy="${PI/10} ${PI/5} 0"/>
+        <parent link="base_link" />
+        <child link="front_left_trans_spring_link" />
+    </joint>
+    <link name="front_right_trans_link">
+        <visual>
+            <origin xyz="0 0 0" rpy="0 0 0"/>
+            <geometry>
+                <cylinder radius="0.02" length="0.28"/>
+            </geometry>
+            <material name="black"/>
+        </visual>
+        <collision>
+            <origin xyz="0 0 0" rpy="0 0 0"/>
+            <geometry>
+                <cylinder radius="0.02" length="0.28"/>
+            </geometry>
+        </collision>
+    </link>
+    <joint name="front_right_trans_joint" type="fixed">
+        <origin xyz="0.15 0.33 0.29" rpy="${PI/10} ${-PI/5} 0"/>
+        <parent link="base_link" />
+        <child link="front_right_trans_link" />
+    </joint>
 </robot>

Commit message: Steps towards ackermann steering

File: kymco_maxxer90_description/urdf/kymco_maxxer90.urdf.xacro (robot description, xacro)
@@ -2,4 +2,5 @@
 <robot name="kymco_maxxer90" xmlns:xacro="http://ros.org/wiki/xacro">
     <xacro:include filename="$(find kymco_maxxer90_description)/urdf/wheel.urdf.xacro"/>
+    <xacro:include filename="$(find kymco_maxxer90_description)/urdf/front_wheel.urdf.xacro"/>
     <xacro:property name="PI" value="3.1415926535897931"/>
     <xacro:property name="distance_from_ground" value="0.35"/> <!-- TODO -->
@@ -25,4 +26,13 @@
         </collision>
     </link>
+    <link name="steering_wheel_link"/>
+    <joint name="steering_wheel_joint" type="revolute">
+        <origin xyz="0 0 0" rpy="0 0 0" />
+        <parent link="base_link" />
+        <child link="steering_wheel_link" />
+        <axis xyz="0 0 1" />
+        <!-- TODO effort and velocity -->
+        <limit lower="${-PI*25/180}" upper="${PI*25/180}" effort="0.5" velocity="4.5"/>
+    </joint>
     <link name="engine_link">
         <visual>
@@ -47,10 +57,10 @@
         <child link="engine_link" />
     </joint>
-    <xacro:kymco_maxxer90_wheel wheel_prefix="front_right">
+    <xacro:kymco_maxxer90_front_wheel wheel_prefix="front_right">
         <origin xyz="${track/2} 0.33 ${distance_from_ground/2}" rpy="0 0 ${PI/2}"/>
-    </xacro:kymco_maxxer90_wheel>
-    <xacro:kymco_maxxer90_wheel wheel_prefix="front_left">
+    </xacro:kymco_maxxer90_front_wheel>
+    <xacro:kymco_maxxer90_front_wheel wheel_prefix="front_left">
         <origin xyz="${-track/2} 0.33 ${distance_from_ground/2}" rpy="0 0 ${-PI/2}"/>
-    </xacro:kymco_maxxer90_wheel>
+    </xacro:kymco_maxxer90_front_wheel>
     <xacro:kymco_maxxer90_wheel wheel_prefix="rear_left">
         <origin xyz="${-track/2} ${0.33-wheelbase} ${distance_from_ground/2}" rpy="0 0 ${-PI/2}"/>
@@ -305,23 +315,3 @@
         <child link="front_left_trans_spring_link" />
     </joint>
-    <link name="front_right_trans_link">
-        <visual>
-            <origin xyz="0 0 0" rpy="0 0 0"/>
-            <geometry>
-                <cylinder radius="0.02" length="0.28"/>
-            </geometry>
-            <material name="black"/>
-        </visual>
-        <collision>
-            <origin xyz="0 0 0" rpy="0 0 0"/>
-            <geometry>
-                <cylinder radius="0.02" length="0.28"/>
-            </geometry>
-        </collision>
-    </link>
-    <joint name="front_right_trans_joint" type="fixed">
-        <origin xyz="0.15 0.33 0.29" rpy="${PI/10} ${-PI/5} 0"/>
-        <parent link="base_link" />
-        <child link="front_right_trans_link" />
-    </joint>
 </robot>

Commit message: STILL trying to have proper inertia simulation

File: kymco_maxxer90_description/urdf/kymco_maxxer90.urdf.xacro (robot description, xacro)
@@ -12,9 +12,4 @@
     <link name="base_link" />
     <link name="chassis_link">
-        <inertial>
-            <mass value="68"/>
-            <origin xyz="-0.08748 -0.00085 0.09947"/>
-                <inertia  ixx="2.746671789898144" ixy="0" ixz="0" iyy="1.629571305145487" iyz="0" izz="1.930434142335272" />
-        </inertial>
         <visual>
             <origin xyz="0 0 ${distance_from_ground}" rpy="0 0 0"/>
@@ -37,4 +32,16 @@
         <parent link="base_link" />"
         <child link="chassis_link" />"
+    </joint>
+    <link name="inertia_link">
+        <inertial>
+            <mass value="68"/>
+            <origin xyz="0 0.2 0.37"/>
+                <inertia  ixx="11.746671789898144" ixy="0" ixz="0" iyy="2.629571305145487" iyz="0" izz="10.930434142335272" />
+        </inertial>
+    </link>
+    <joint name="inertia_joint" type="fixed" >
+        <origin xyz="0 0 0" rpy="0 0 0"/>
+        <parent link="base_link"/>
+        <child link="inertia_link"/>
     </joint>
     <gazebo reference="chassis_link">
@@ -78,10 +85,10 @@
             </material>
         </visual>
-        <collision>
-            <origin xyz="0 0 0" rpy="0 0 0"/>
-            <geometry>
-                <mesh filename="package://kymco_maxxer90_description/meshes/engine.stl" scale="1.0 1.0 1.0"/>
-            </geometry>
-        </collision>
+        <!-- <collision> -->
+            <!-- <origin xyz="0 0 0" rpy="0 0 0"/> -->
+            <!-- <geometry> -->
+                <!-- <mesh filename="package://kymco_maxxer90_description/meshes/engine.stl" scale="1.0 1.0 1.0"/> -->
+            <!-- </geometry> -->
+        <!-- </collision> -->
     </link>
     <joint name="engine_joint" type="fixed">
@@ -94,16 +101,16 @@
     </gazebo>"
     <!-- Wheels -->
-    <xacro:kymco_maxxer90_front_wheel wheel_prefix="front_right">
-        <origin xyz="${track/2} 0.33 ${distance_from_ground/2}" rpy="0 0 ${PI/2}"/>
-    </xacro:kymco_maxxer90_front_wheel>
-    <xacro:kymco_maxxer90_front_wheel wheel_prefix="front_left">
-        <origin xyz="${-track/2} 0.33 ${distance_from_ground/2}" rpy="0 0 ${-PI/2}"/>
-    </xacro:kymco_maxxer90_front_wheel>
-    <xacro:kymco_maxxer90_wheel wheel_prefix="rear_left">
-        <origin xyz="${-track/2} ${0.33-wheelbase} ${distance_from_ground/2}" rpy="0 0 ${-PI/2}"/>
-    </xacro:kymco_maxxer90_wheel>
-    <xacro:kymco_maxxer90_wheel wheel_prefix="rear_right">
-        <origin xyz="${track/2} ${0.33-wheelbase} ${distance_from_ground/2}" rpy="0 0 ${PI/2}"/>
-    </xacro:kymco_maxxer90_wheel>
+    <!-- <xacro:kymco_maxxer90_front_wheel wheel_prefix="front_right"> -->
+        <!-- <origin xyz="${track/2} 0.33 ${distance_from_ground/2}" rpy="0 0 ${PI/2}"/> -->
+    <!-- </xacro:kymco_maxxer90_front_wheel> -->
+    <!-- <xacro:kymco_maxxer90_front_wheel wheel_prefix="front_left"> -->
+        <!-- <origin xyz="${-track/2} 0.33 ${distance_from_ground/2}" rpy="0 0 ${-PI/2}"/> -->
+    <!-- </xacro:kymco_maxxer90_front_wheel> -->
+    <!-- <xacro:kymco_maxxer90_wheel wheel_prefix="rear_left"> -->
+        <!-- <origin xyz="${-track/2} ${0.33-wheelbase} ${distance_from_ground/2}" rpy="0 0 ${-PI/2}"/> -->
+    <!-- </xacro:kymco_maxxer90_wheel> -->
+    <!-- <xacro:kymco_maxxer90_wheel wheel_prefix="rear_right"> -->
+        <!-- <origin xyz="${track/2} ${0.33-wheelbase} ${distance_from_ground/2}" rpy="0 0 ${PI/2}"/> -->
+    <!-- </xacro:kymco_maxxer90_wheel> -->
     <link name="rear_axle_link">
         <visual>
@@ -114,10 +121,10 @@
             <material name="silver"/>
         </visual>
-        <collision>
-            <origin xyz="0 0 0" rpy="0 0 0"/>
-            <geometry>
-                <mesh filename="package://kymco_maxxer90_description/meshes/differential.stl" scale="1.0 1.0 1.0"/>
-            </geometry>
-        </collision>
+        <!-- <collision> -->
+            <!-- <origin xyz="0 0 0" rpy="0 0 0"/> -->
+            <!-- <geometry> -->
+                <!-- <mesh filename="package://kymco_maxxer90_description/meshes/differential.stl" scale="1.0 1.0 1.0"/> -->
+            <!-- </geometry> -->
+        <!-- </collision> -->
     </link>
     <joint name="rear_axle_joint" type="fixed">
@@ -137,10 +144,10 @@
             <material name="silver"/>
         </visual>
-        <collision>
-            <origin xyz="0 0 0" rpy="0 0 0"/>
-            <geometry>
-                <box size="0.4 0.3 0.01"/>
-            </geometry>
-        </collision>
+        <!-- <collision> -->
+            <!-- <origin xyz="0 0 0" rpy="0 0 0"/> -->
+            <!-- <geometry> -->
+                <!-- <box size="0.4 0.3 0.01"/> -->
+            <!-- </geometry> -->
+        <!-- </collision> -->
     </link>
     <joint name="front_plate_joint" type="fixed">
@@ -160,10 +167,10 @@
             <material name="silver"/>
         </visual>
-        <collision>
-            <origin xyz="0 0 0" rpy="0 0 0"/>
-            <geometry>
-                <box size="0.4 0.3 0.01"/>
-            </geometry>
-        </collision>
+        <!-- <collision> -->
+            <!-- <origin xyz="0 0 0" rpy="0 0 0"/> -->
+            <!-- <geometry> -->
+                <!-- <box size="0.4 0.3 0.01"/> -->
+            <!-- </geometry> -->
+        <!-- </collision> -->
     </link>
     <joint name="rear_plate_joint" type="fixed">
@@ -183,10 +190,10 @@
             <material name="black"/>
         </visual>
-        <collision>
-            <origin xyz="0 0 0" rpy="0 0 0"/>
-            <geometry>
-                <box size="0.12 0.01 0.01"/>
-            </geometry>
-        </collision>
+        <!-- <collision> -->
+            <!-- <origin xyz="0 0 0" rpy="0 0 0"/> -->
+            <!-- <geometry> -->
+                <!-- <box size="0.12 0.01 0.01"/> -->
+            <!-- </geometry> -->
+        <!-- </collision> -->
     </link>
     <joint name="rear_trans_chassis_joint" type="fixed">
@@ -206,10 +213,10 @@
             <material name="black"/>
         </visual>
-        <collision>
-            <origin xyz="0 0 0" rpy="0 0 0"/>
-            <geometry>
-                <cylinder radius="0.02" length="0.28"/>
-            </geometry>
-        </collision>
+        <!-- <collision> -->
+            <!-- <origin xyz="0 0 0" rpy="0 0 0"/> -->
+            <!-- <geometry> -->
+                <!-- <cylinder radius="0.02" length="0.28"/> -->
+            <!-- </geometry> -->
+        <!-- </collision> -->
     </link>
     <joint name="rear_trans_joint" type="fixed">
@@ -231,10 +238,10 @@
             </material>
         </visual>
-        <collision>
-            <origin xyz="0 0 0" rpy="0 0 0"/>
-            <geometry>
-                <mesh filename="package://kymco_maxxer90_description/meshes/spring.stl" scale="1.0 1.0 1.0"/>
-            </geometry>
-        </collision>
+        <!-- <collision> -->
+            <!-- <origin xyz="0 0 0" rpy="0 0 0"/> -->
+            <!-- <geometry> -->
+                <!-- <mesh filename="package://kymco_maxxer90_description/meshes/spring.stl" scale="1.0 1.0 1.0"/> -->
+            <!-- </geometry> -->
+        <!-- </collision> -->
     </link>
     <gazebo reference="rear_trans_spring_link">
@@ -254,10 +261,10 @@
             <material name="black"/>
         </visual>
-        <collision>
-            <origin xyz="0 0 0" rpy="0 0 0"/>
-            <geometry>
-                <box size="0.01 0.2 0.01"/>
-            </geometry>
-        </collision>
+        <!-- <collision> -->
+            <!-- <origin xyz="0 0 0" rpy="0 0 0"/> -->
+            <!-- <geometry> -->
+                <!-- <box size="0.01 0.2 0.01"/> -->
+            <!-- </geometry> -->
+        <!-- </collision> -->
     </link>
     <joint name="front_right_trans_chassis_joint" type="fixed">
@@ -277,10 +284,10 @@
             <material name="black"/>
         </visual>
-        <collision>
-            <origin xyz="0 0 0" rpy="0 0 0"/>
-            <geometry>
-                <cylinder radius="0.02" length="0.28"/>
-            </geometry>
-        </collision>
+        <!-- <collision> -->
+            <!-- <origin xyz="0 0 0" rpy="0 0 0"/> -->
+            <!-- <geometry> -->
+                <!-- <cylinder radius="0.02" length="0.28"/> -->
+            <!-- </geometry> -->
+        <!-- </collision> -->
     </link>
     <joint name="front_right_trans_joint" type="fixed">
@@ -302,10 +309,10 @@
             </material>
         </visual>
-        <collision>
-            <origin xyz="0 0 0" rpy="0 0 0"/>
-            <geometry>
-                <mesh filename="package://kymco_maxxer90_description/meshes/spring.stl" scale="1.0 1.0 1.0"/>
-            </geometry>
-        </collision>
+        <!-- <collision> -->
+            <!-- <origin xyz="0 0 0" rpy="0 0 0"/> -->
+            <!-- <geometry> -->
+                <!-- <mesh filename="package://kymco_maxxer90_description/meshes/spring.stl" scale="1.0 1.0 1.0"/> -->
+            <!-- </geometry> -->
+        <!-- </collision> -->
     </link>
     <joint name="front_right_trans_spring_joint" type="fixed">
@@ -325,10 +332,10 @@
             <material name="black"/>
         </visual>
-        <collision>
-            <origin xyz="0 0 0" rpy="0 0 0"/>
-            <geometry>
-                <box size="0.01 0.2 0.01"/>
-            </geometry>
-        </collision>
+        <!-- <collision> -->
+            <!-- <origin xyz="0 0 0" rpy="0 0 0"/> -->
+            <!-- <geometry> -->
+                <!-- <box size="0.01 0.2 0.01"/> -->
+            <!-- </geometry> -->
+        <!-- </collision> -->
     </link>
     <joint name="front_left_trans_chassis_joint" type="fixed">
@@ -348,10 +355,10 @@
             <material name="black"/>
         </visual>
-        <collision>
-            <origin xyz="0 0 0" rpy="0 0 0"/>
-            <geometry>
-                <cylinder radius="0.02" length="0.28"/>
-            </geometry>
-        </collision>
+        <!-- <collision> -->
+            <!-- <origin xyz="0 0 0" rpy="0 0 0"/> -->
+            <!-- <geometry> -->
+                <!-- <cylinder radius="0.02" length="0.28"/> -->
+            <!-- </geometry> -->
+        <!-- </collision> -->
     </link>
     <joint name="front_left_trans_joint" type="fixed">
@@ -373,10 +380,10 @@
             </material>
         </visual>
-        <collision>
-            <origin xyz="0 0 0" rpy="0 0 0"/>
-            <geometry>
-                <mesh filename="package://kymco_maxxer90_description/meshes/spring.stl" scale="1.0 1.0 1.0"/>
-            </geometry>
-        </collision>
+        <!-- <collision> -->
+            <!-- <origin xyz="0 0 0" rpy="0 0 0"/> -->
+            <!-- <geometry> -->
+                <!-- <mesh filename="package://kymco_maxxer90_description/meshes/spring.stl" scale="1.0 1.0 1.0"/> -->
+            <!-- </geometry> -->
+        <!-- </collision> -->
     </link>
     <joint name="front_left_trans_spring_joint" type="fixed">
