Commit message: First kinda-working version of the rear suspension

File: kymco_maxxer90_description/urdf/kymco_maxxer90.urdf.xacro (robot description, xacro)
@@ -113,4 +113,25 @@
         <origin xyz="${track/2} 0 0" rpy="0 0 ${PI/2}"/>
     </xacro:kymco_maxxer90_wheel>
+    <link name="rear_suspension_link" >
+        <inertial>
+            <mass value="1"/>
+            <origin xyz="0 0 0"/>
+            <inertia ixx="0.01" ixy="0" ixz="0" iyy="0.01" iyz="0" izz="0.01"/>
+        </inertial>
+    </link>
+    <joint name="rear_suspension_joint" type="prismatic">
+        <origin xyz="0 ${0.33-wheelbase} ${distance_from_ground/2}" rpy="0 0 0" />
+        <parent link="base_link"/>
+        <child link="rear_suspension_link"/>
+        <axis xyz="0 0 -1" />
+        <limit lower="-0.1" upper="0.1" effort="500" velocity="10"/>
+        <!-- <dynamics damping="1" friction="0.2"/> -->
+    </joint>
+    <gazebo reference="rear_suspension_joint">
+        <provideFeedback>true</provideFeedback>
+        <implicitSpringDamper>true</implicitSpringDamper>
+        <springStiffness>30000</springStiffness>
+        <springReference>0</springReference>
+    </gazebo>
     <link name="rear_axle_link">
         <visual>
@@ -129,6 +150,6 @@
     </link>
     <joint name="rear_axle_joint" type="fixed">
-        <origin xyz="0.03 ${0.33-wheelbase} ${distance_from_ground/2}" rpy="0 0 ${-PI/2}"/>
-        <parent link="base_link" />
+        <origin xyz="0.03 0 0" rpy="0 0 ${-PI/2}"/>
+        <parent link="rear_suspension_link" />
         <child link="rear_axle_link" />
     </joint>
@@ -138,5 +159,5 @@
     <link name="RWD">
         <inertial>
-            <mass value="5"/>
+            <mass value="1"/>
             <origin xyz="0 0 0"/>
             <inertia ixx="0.01" ixy="0" ixz="0" iyy="0.01" iyz="0" izz="0.01"/>
@@ -144,6 +165,6 @@
     </link>
     <joint name="RWD_joint" type="continuous">
-        <origin xyz="0 ${0.33-wheelbase} ${distance_from_ground/2}" rpy="0 0 0"/>
-        <parent link="base_link" />
+        <origin xyz="0 0 0" rpy="0 0 0"/>
+        <parent link="rear_suspension_link" />
         <child link="RWD" />
         <axis xyz="-1 0 0" />

Commit message: More precise steering velocity and sane inertia

File: kymco_maxxer90_description/urdf/kymco_maxxer90.urdf.xacro (robot description, xacro)
@@ -51,17 +51,17 @@
     <link name="steering_wheel_link">
         <inertial>
-            <mass value="1"/>
+            <mass value="0.01"/>
             <origin xyz="0 0 0"/>
-            <inertia ixx="0.01" ixy="0" ixz="0" iyy="0.01" iyz="0" izz="0.01"/>
+            <inertia ixx="0.0001" ixy="0" ixz="0" iyy="0.0001" iyz="0" izz="0.0001"/>
         </inertial>
     </link>
     <joint name="steering_wheel_joint" type="revolute">
-        <origin xyz="0 0 0" rpy="0 0 0" />
+        <origin xyz="0 0.33 ${distance_from_ground}" rpy="0 0 0" />
         <parent link="base_link" />
         <child link="steering_wheel_link" />
         <axis xyz="0 0 1" />
         <!-- TODO effort and velocity -->
-        <limit lower="${-PI*25/180}" upper="${PI*25/180}" effort="100.5" velocity="4.5"/>
-        <dynamics damping="3" friction="0.0" />
+        <limit lower="${-PI*25/180}" upper="${PI*25/180}" effort="100000" velocity="0.95"/>
+        <dynamics damping="0" friction="0.0" />
     </joint>
     <transmission name="steering_wheel_joint_trans">

Commit message: Added simulated rgbd camera

File: kymco_maxxer90_description/urdf/kymco_maxxer90.urdf.xacro (robot description, xacro)
@@ -459,4 +459,57 @@
         <child link="imu_link"/>
     </joint>
+    <link name="rgbd_optical_camera_frame"/>
+    <joint name="rgbd_optical_camera_joint" type="fixed">
+        <origin xyz="0.0 0.5 0.4" rpy="0 0 ${PI/2}"/>
+        <parent link="base_link"/>
+        <child link="rgbd_optical_camera_frame"/>
+    </joint>
+    <link name="rgbd_depth_camera_frame"/>
+    <joint name="rgbd_depth_camera_joint" type="fixed">
+        <origin xyz="0.0 0 0" rpy="${-PI/2} 0 ${-PI/2}"/>
+        <parent link="rgbd_optical_camera_frame"/>
+        <child link="rgbd_depth_camera_frame"/>
+    </joint>
+    <gazebo reference="rgbd_optical_camera_frame">
+        <sensor type="depth" name="camera">
+            <always_on>true</always_on>
+            <update_rate>30.0</update_rate>
+            <camera>
+                <horizontal_fov>${110.0*PI/180.0}</horizontal_fov>
+                <image>
+                    <format>R8G8B8</format>
+                    <width>720</width>
+                    <height>540</height>
+                </image>
+                <clip>
+                    <near>0.2</near>
+                    <far>10.0</far>
+                </clip>
+            </camera>
+            <plugin name="camera_plugin" filename="libgazebo_ros_openni_kinect.so">
+                <baseline>0.2</baseline>
+                <alwaysOn>true</alwaysOn>
+                <!-- <cameraName>camera_ir</cameraName> -->
+                <imageTopicName>/camera/color/image_raw</imageTopicName>
+                <cameraInfoTopicName>/camera/color/camera_info</cameraInfoTopicName>
+                <depthImageTopicName>/camera/depth/image_raw</depthImageTopicName>
+                <depthImageCameraInfoTopicName>/camera/depth/camera_info</depthImageCameraInfoTopicName>
+                <pointCloudTopicName>/camera/depth/points</pointCloudTopicName>
+                <frameName>rgbd_depth_camera_frame</frameName>
+                <pointCloudCutoff>0.2</pointCloudCutoff>
+                <pointCloudCutoffMax>10.0</pointCloudCutoffMax>
+                <distortionK1>-0.16</distortionK1>
+                <distortionK2>0.01</distortionK2>
+                <distortionK3>-0.02</distortionK3>
+                <distortionT1>0.004</distortionT1>
+                <distortionT2>-0.01</distortionT2>
+                <CxPrime>0</CxPrime>
+                <Cx>0</Cx>
+                <Cy>0</Cy>
+                <focalLength>0</focalLength>
+                <hackBaseline>0</hackBaseline>
+            </plugin>
+        </sensor>
+    </gazebo>
     <!-- Gazebo plugins -->
     <gazebo>

Commit message: Model revisited. (Almost) EVERYTHING has been changed. I need to check some stuff again.

File: kymco_maxxer90_description/urdf/kymco_maxxer90.urdf.xacro (robot description, xacro)
@@ -8,8 +8,13 @@
     <xacro:property name="wheel_diameter" value="0.4572"/>
     <xacro:property name="wheel_width" value="0.15"/>
-    <xacro:property name="track" value="0.55"/>
+    <xacro:property name="track" value="0.835"/>
     <!-- Chassis -->
     <link name="base_link" />
     <link name="chassis_link">
+        <inertial>
+            <mass value="68"/>
+            <origin xyz="-0.25 0 ${distance_from_ground}" rpy="0 0 0"/>
+            <inertia  ixx="6.997767154121414" ixy="0" ixz="0" iyy="17.876069102859596" iyz="0" izz="18.49883625698101" />
+        </inertial>
         <visual>
             <origin xyz="0 0 ${distance_from_ground}" rpy="0 0 0"/>
@@ -33,16 +38,4 @@
         <child link="chassis_link" />"
     </joint>
-    <link name="inertia_link">
-        <inertial>
-            <mass value="68"/>
-            <origin xyz="0 -0.2 0.37"/>
-                <inertia  ixx="11.746671789898144" ixy="0" ixz="0" iyy="2.629571305145487" iyz="0" izz="10.930434142335272" />
-        </inertial>
-    </link>
-    <joint name="inertia_joint" type="fixed" >
-        <origin xyz="0 0 0" rpy="0 0 0"/>
-        <parent link="base_link"/>
-        <child link="inertia_link"/>
-    </joint>
     <gazebo reference="chassis_link">
         <material>Gazebo/Black</material>
@@ -51,5 +44,5 @@
     <link name="steering_wheel_link">
         <inertial>
-            <mass value="20"/>
+            <mass value="2"/>
             <origin xyz="0 0 0"/>
             <inertia ixx="0.0001" ixy="0" ixz="0" iyy="0.0001" iyz="0" izz="0.0001"/>
@@ -57,5 +50,5 @@
     </link>
     <joint name="steering_wheel_joint" type="revolute">
-        <origin xyz="0 0.33 ${distance_from_ground}" rpy="0 0 0" />
+        <origin xyz="0 0 0" rpy="0 0 0" />
         <parent link="base_link" />
         <child link="steering_wheel_link" />
@@ -78,5 +71,5 @@
             <origin xyz="0 0 0" rpy="0 0 0"/>
             <geometry>
-                <mesh filename="package://kymco_maxxer90_description/meshes/engine.stl" scale="1.0 1.0 1.0"/>
+                <mesh filename="package://kymco_maxxer90_description/meshes/engine.stl" scale="1.3 1.3 1.3"/>
             </geometry>
             <material name="silver">
@@ -87,10 +80,10 @@
             <origin xyz="0 0 0" rpy="0 0 0"/>
             <geometry>
-                <mesh filename="package://kymco_maxxer90_description/meshes/engine.stl" scale="1.0 1.0 1.0"/>
+                <mesh filename="package://kymco_maxxer90_description/meshes/engine.stl" scale="1.3 1.3 1.3"/>
             </geometry>
         </collision>
     </link>
     <joint name="engine_joint" type="fixed">
-        <origin xyz="0 -0.08 ${distance_from_ground+0.05}" rpy="0 0 ${PI/2}"/>
+        <origin xyz="-0.08 0 ${distance_from_ground+0.05}" rpy="0 0 0"/>
         <parent link="base_link" />
         <child link="engine_link" />
@@ -101,14 +94,14 @@
     <!-- Wheels -->
     <xacro:kymco_maxxer90_front_wheel wheel_prefix="front_right">
-        <origin xyz="${track/2} 0.33 ${distance_from_ground/2}" rpy="0 0 ${PI/2}"/>
+        <origin xyz="0.33 ${track/2} ${distance_from_ground/2}" rpy="0 0 ${PI}"/>
     </xacro:kymco_maxxer90_front_wheel>
     <xacro:kymco_maxxer90_front_wheel wheel_prefix="front_left">
-        <origin xyz="${-track/2} 0.33 ${distance_from_ground/2}" rpy="0 0 ${-PI/2}"/>
+        <origin xyz="0.33 ${-track/2} ${distance_from_ground/2}" rpy="0 0 0"/>
     </xacro:kymco_maxxer90_front_wheel>
+    <xacro:kymco_maxxer90_wheel wheel_prefix="rear_right">
+        <origin xyz="0 ${track/2} 0" rpy="0 0 ${PI}"/>
+    </xacro:kymco_maxxer90_wheel>
     <xacro:kymco_maxxer90_wheel wheel_prefix="rear_left">
-        <origin xyz="${-track/2} 0 0" rpy="0 0 ${-PI/2}"/>
-    </xacro:kymco_maxxer90_wheel>
-    <xacro:kymco_maxxer90_wheel wheel_prefix="rear_right">
-        <origin xyz="${track/2} 0 0" rpy="0 0 ${PI/2}"/>
+        <origin xyz="0 ${-track/2} 0" rpy="0 0 0"/>
     </xacro:kymco_maxxer90_wheel>
     <link name="rear_suspension_link" >
@@ -120,5 +113,5 @@
     </link>
     <joint name="rear_suspension_joint" type="prismatic">
-        <origin xyz="0 ${0.33-wheelbase} ${distance_from_ground/2}" rpy="0 0 0" />
+        <origin xyz="${0.33-wheelbase} 0 ${distance_from_ground/2}" rpy="0 0 0" />
         <parent link="base_link"/>
         <child link="rear_suspension_link"/>
@@ -144,19 +137,19 @@
     <link name="rear_axle_link">
         <visual>
-            <origin xyz="0 0 0" rpy="0 0 0"/>
-            <geometry>
-                <mesh filename="package://kymco_maxxer90_description/meshes/differential.stl" scale="1.0 1.0 1.0"/>
+            <origin xyz="0 0.05 0" rpy="0 0 0"/>
+            <geometry>
+                <mesh filename="package://kymco_maxxer90_description/meshes/differential.stl" scale="1.6 1.6 1.6"/>
             </geometry>
             <material name="silver"/>
         </visual>
         <collision>
-            <origin xyz="0 0 0" rpy="0 0 0"/>
-            <geometry>
-                <mesh filename="package://kymco_maxxer90_description/meshes/differential.stl" scale="1.0 1.0 1.0"/>
+            <origin xyz="0 0.05 0" rpy="0 0 0"/>
+            <geometry>
+                <mesh filename="package://kymco_maxxer90_description/meshes/differential.stl" scale="1.6 1.6 1.6"/>
             </geometry>
         </collision>
     </link>
     <joint name="rear_axle_joint" type="fixed">
-        <origin xyz="0.03 0 0" rpy="0 0 ${-PI/2}"/>
+        <origin xyz="0 0 0" rpy="0 0 0"/>
         <parent link="rear_suspension_link" />
         <child link="rear_axle_link" />
@@ -176,5 +169,5 @@
         <parent link="rear_suspension_link" />
         <child link="RWD" />
-        <axis xyz="-1 0 0" />
+        <axis xyz="0 1 0" />
     </joint>
     <transmission name="non_differential_trans" type="SimpleTransmission">
@@ -191,5 +184,5 @@
             <origin xyz="0 0 0" rpy="0 0 0"/>
             <geometry>
-                <box size="0.4 0.3 0.01"/>
+                <box size="0.3 0.4 0.01"/>
             </geometry>
             <material name="silver"/>
@@ -198,10 +191,10 @@
             <origin xyz="0 0 0" rpy="0 0 0"/>
             <geometry>
-                <box size="0.4 0.3 0.01"/>
+                <box size="0.3 0.4 0.01"/>
             </geometry>
         </collision>
     </link>
     <joint name="front_plate_joint" type="fixed">
-        <origin xyz="0 0.45 0.561" rpy="0 0 0"/>
+        <origin xyz="0.33 0 0.65" rpy="0 0 0"/>
         <parent link="base_link" />
         <child link="front_plate_link" />
@@ -214,5 +207,5 @@
             <origin xyz="0 0 0" rpy="0 0 0"/>
             <geometry>
-                <box size="0.4 0.3 0.01"/>
+                <box size="0.3 0.4 0.01"/>
             </geometry>
             <material name="silver"/>
@@ -221,10 +214,10 @@
             <origin xyz="0 0 0" rpy="0 0 0"/>
             <geometry>
-                <box size="0.4 0.3 0.01"/>
+                <box size="0.3 0.4 0.01"/>
             </geometry>
         </collision>
     </link>
     <joint name="rear_plate_joint" type="fixed">
-        <origin xyz="0 -0.66 0.59" rpy="${-PI/13} 0 0"/>
+        <origin xyz="-0.75 0 0.67" rpy="0 ${PI/13} 0"/>
         <parent link="base_link" />
         <child link="rear_plate_link" />
@@ -237,5 +230,5 @@
             <origin xyz="0 0 0" rpy="0 0 0"/>
             <geometry>
-                <box size="0.12 0.01 0.01"/>
+                <box size="0.02 0.22 0.02"/>
             </geometry>
             <material name="black"/>
@@ -244,10 +237,10 @@
             <origin xyz="0 0 0" rpy="0 0 0"/>
             <geometry>
-                <box size="0.12 0.01 0.01"/>
+                <box size="0.02 0.22 0.02"/>
             </geometry>
         </collision>
     </link>
     <joint name="rear_trans_chassis_joint" type="fixed">
-        <origin xyz="0 -0.46 0.39" rpy="0 0 0"/>
+        <origin xyz="-0.57 0 0.48" rpy="0 0 0"/>
         <parent link="base_link" />
         <child link="rear_trans_chassis_link" />
@@ -272,5 +265,5 @@
     </link>
     <joint name="rear_trans_joint" type="fixed">
-        <origin xyz="0 -0.56 0.29" rpy="${-PI/4} 0 0"/>
+        <origin xyz="-0.6 0 0.34" rpy="0 ${PI/16} 0"/>
         <parent link="base_link" />
         <child link="rear_trans_link" />
@@ -300,5 +293,5 @@
     </gazebo>"
     <joint name="rear_trans_spring_joint" type="fixed">
-        <origin xyz="0 -0.56 0.29" rpy="${-PI/4} 0 0"/>
+        <origin xyz="-0.6 0 0.34" rpy="0 ${PI/16} 0"/>
         <parent link="base_link" />
         <child link="rear_trans_spring_link" />
@@ -308,5 +301,5 @@
             <origin xyz="0 0 0" rpy="0 0 0"/>
             <geometry>
-                <box size="0.01 0.2 0.01"/>
+                <box size="0.3 0.02 0.01"/>
             </geometry>
             <material name="black"/>
@@ -315,10 +308,10 @@
             <origin xyz="0 0 0" rpy="0 0 0"/>
             <geometry>
-                <box size="0.01 0.2 0.01"/>
+                <box size="0.3 0.02 0.01"/>
             </geometry>
         </collision>
     </link>
     <joint name="front_right_trans_chassis_joint" type="fixed">
-        <origin xyz="0.075 0.33 0.4" rpy="0 0 0"/>
+        <origin xyz="0.33 0.16 0.4" rpy="0 0 0"/>
         <parent link="base_link" />
         <child link="front_right_trans_chassis_link" />
@@ -343,5 +336,5 @@
     </link>
     <joint name="front_right_trans_joint" type="fixed">
-        <origin xyz="0.15 0.33 0.29" rpy="${PI/10} ${-PI/5} 0"/>
+        <origin xyz="0.33 0.25 0.29" rpy="${PI/5} ${-PI/10} 0"/>
         <parent link="base_link" />
         <child link="front_right_trans_link" />
@@ -368,5 +361,5 @@
     </link>
     <joint name="front_right_trans_spring_joint" type="fixed">
-        <origin xyz="0.15 0.33 0.29" rpy="${PI/10} ${-PI/5} 0"/>
+        <origin xyz="0.33 0.25 0.29" rpy="${PI/5} ${-PI/10} 0"/>
         <parent link="base_link" />
         <child link="front_right_trans_spring_link" />
@@ -379,5 +372,5 @@
             <origin xyz="0 0 0" rpy="0 0 0"/>
             <geometry>
-                <box size="0.01 0.2 0.01"/>
+                <box size="0.3 0.02 0.01"/>
             </geometry>
             <material name="black"/>
@@ -386,10 +379,10 @@
             <origin xyz="0 0 0" rpy="0 0 0"/>
             <geometry>
-                <box size="0.01 0.2 0.01"/>
+                <box size="0.3 0.02 0.01"/>
             </geometry>
         </collision>
     </link>
     <joint name="front_left_trans_chassis_joint" type="fixed">
-        <origin xyz="-0.075 0.33 0.4" rpy="0 0 0"/>
+        <origin xyz="0.33 -0.16 0.4" rpy="0 0 0"/>
         <parent link="base_link" />
         <child link="front_left_trans_chassis_link" />
@@ -414,5 +407,5 @@
     </link>
     <joint name="front_left_trans_joint" type="fixed">
-        <origin xyz="-0.15 0.33 0.29" rpy="${PI/10} ${PI/5} 0"/>
+        <origin xyz="0.33 -0.25 0.29" rpy="${-PI/5} ${-PI/10} 0"/>
         <parent link="base_link" />
         <child link="front_left_trans_link" />
@@ -439,5 +432,5 @@
     </link>
     <joint name="front_left_trans_spring_joint" type="fixed">
-        <origin xyz="-0.15 0.33 0.29" rpy="${PI/10} ${PI/5} 0"/>
+        <origin xyz="0.33 -0.25 0.29" rpy="${-PI/5} ${-PI/10} 0"/>
         <parent link="base_link" />
         <child link="front_left_trans_spring_link" />
@@ -461,5 +454,5 @@
     <link name="rgbd_optical_camera_frame"/>
     <joint name="rgbd_optical_camera_joint" type="fixed">
-        <origin xyz="0.0 0.5 0.4" rpy="0 0 ${PI/2}"/>
+        <origin xyz="0.5 0.0 0.4" rpy="0 0 ${PI/2}"/>
         <parent link="base_link"/>
         <child link="rgbd_optical_camera_frame"/>
@@ -514,5 +507,5 @@
     <!-- Gazebo plugins -->
     <gazebo>
-        <plugin name="gps_controller" filename="libhector_gazebo_ros_gps.so">
+        <plugin name="gps_sensor" filename="libhector_gazebo_ros_gps.so">
             <robotNamespace>/</robotNamespace>
             <updateRate>40</updateRate>
@@ -527,5 +520,5 @@
             <drift>0.0001 0.0001 0.0001</drift>
         </plugin>
-        <plugin name="jaguar_imu_sensor" filename="libhector_gazebo_ros_imu.so">
+        <plugin name="imu_sensor" filename="libhector_gazebo_ros_imu.so">
             <updateRate>50.0</updateRate>
             <bodyName>base_link</bodyName>

Commit message: Fixed gps frame and camera orientation

File: kymco_maxxer90_description/urdf/kymco_maxxer90.urdf.xacro (robot description, xacro)
@@ -454,5 +454,5 @@
     <link name="rgbd_optical_camera_frame"/>
     <joint name="rgbd_optical_camera_joint" type="fixed">
-        <origin xyz="0.5 0.0 0.4" rpy="0 0 ${PI/2}"/>
+        <origin xyz="0.5 0.0 0.4" rpy="0 0 0"/>
         <parent link="base_link"/>
         <child link="rgbd_optical_camera_frame"/>
@@ -511,5 +511,5 @@
             <updateRate>40</updateRate>
             <bodyName>base_link</bodyName>
-            <frameId>base_link</frameId>
+            <frameId>gps_link</frameId>
             <topicName>navsat/fix</topicName>
             <velocityTopicName>navsat/vel</velocityTopicName>

Commit message: Added camera_link as root for the camera sensor

File: kymco_maxxer90_description/urdf/kymco_maxxer90.urdf.xacro (robot description, xacro)
@@ -452,8 +452,14 @@
         <child link="imu_link"/>
     </joint>
+    <link name="camera_link"/>
+    <joint name="camera_joint" type="fixed">
+        <origin xyz="0.5 0.0 0.4" rpy="0 0 0"/>
+        <parent link="base_link"/>
+        <child link="camera_link"/>
+    </joint>
     <link name="rgbd_optical_camera_frame"/>
     <joint name="rgbd_optical_camera_joint" type="fixed">
-        <origin xyz="0.5 0.0 0.4" rpy="0 0 0"/>
-        <parent link="base_link"/>
+        <origin xyz="0 0 0" rpy="0 0 0"/>
+        <parent link="camera_link"/>
         <child link="rgbd_optical_camera_frame"/>
     </joint>

Commit message: Fixed camera position based on the real scenario

File: kymco_maxxer90_description/urdf/kymco_maxxer90.urdf.xacro (robot description, xacro)
@@ -454,5 +454,5 @@
     <link name="camera_link"/>
     <joint name="camera_joint" type="fixed">
-        <origin xyz="0.5 0.0 0.4" rpy="0 0 0"/>
+        <origin xyz="0.5 0.0 0.63" rpy="0 -0.15 0"/>
         <parent link="base_link"/>
         <child link="camera_link"/>

Commit message: Added the usb cam and an extra link for the position of the spraying valve

File: kymco_maxxer90_description/urdf/kymco_maxxer90.urdf.xacro (robot description, xacro)
@@ -223,4 +223,10 @@
         <child link="rear_plate_link" />
     </joint>
+    <link name="spray_valve_link"/>
+    <joint name="spray_valve_joint" type="fixed">
+        <origin xyz="-0.7 0.2 0.9" rpy="0 0 1.57079632679"/>
+        <parent link="base_link" />
+        <child link="spray_valve_link" />
+    </joint>
     <gazebo reference="rear_plate_link">
         <material>Gazebo/Grey</material>
@@ -457,4 +463,10 @@
         <parent link="base_link"/>
         <child link="camera_link"/>
+    </joint>
+    <link name="webcamera_link"/>
+    <joint name="webcamera_joint" type="fixed">
+        <origin xyz="0.4 0.15 0.69" rpy="0 0 0.2"/>
+        <parent link="base_link"/>
+        <child link="webcamera_link"/>
     </joint>
     <link name="rgbd_optical_camera_frame"/>
@@ -511,4 +523,40 @@
         </sensor>
     </gazebo>
+    <gazebo reference="webcamera_link">
+    <sensor type="camera" name="webcam">
+      <update_rate>30.0</update_rate>
+      <camera name="usb_cam">
+        <horizontal_fov>1.3962634</horizontal_fov>
+        <image>
+          <width>640</width>
+          <height>480</height>
+          <format>R8G8B8</format>
+        </image>
+        <clip>
+          <near>0.02</near>
+          <far>100</far>
+        </clip>
+        <noise>
+          <type>gaussian</type>
+          <mean>0.0</mean>
+          <stddev>0.007</stddev>
+        </noise>
+      </camera>
+      <plugin name="camera_controller" filename="libgazebo_ros_camera.so">
+        <alwaysOn>true</alwaysOn>
+        <updateRate>0.0</updateRate>
+        <cameraName>usb_cam</cameraName>
+        <imageTopicName>image_raw</imageTopicName>
+        <cameraInfoTopicName>camera_info</cameraInfoTopicName>
+        <frameName>webcamera_link</frameName>
+        <hackBaseline>0.07</hackBaseline>
+        <distortionK1>0.0</distortionK1>
+        <distortionK2>0.0</distortionK2>
+        <distortionK3>0.00</distortionK3>
+        <distortionT1>0.00</distortionT1>
+        <distortionT2>0.000</distortionT2>
+      </plugin>
+    </sensor>
+  </gazebo>
     <!-- Gazebo plugins -->
     <gazebo>
